File: hardware/mainboard/chartreuse/chartreuse-usb.sch (KiCad schematic (older format))
At the start: 0 parts

Commit message: Finish HDMI circuit (mostly)
Added most of the connections and minor components in the HDMI sheet. In addition, added the USB hub IC to the USB sheet.
Parts:
- added C?: C_Small, symbol Device:C_Small
- added L?: Ferrite_Bead_Small, symbol Device:Ferrite_Bead_Small
- added U?: USB2422, symbol chartreuse:USB2422
Connections:
- net labels added: GND
- wire segments 0 -> 19
Changed lines of the file:
@@
 Comment4 ""
 $EndDescr
-Text HLabel 4800 3000 0    50   Input ~ 0
+Text HLabel 5200 3500 0    50   Input ~ 0
 USB_UP_DP
-Text HLabel 4800 3100 0    50   Input ~ 0
+Text HLabel 5200 3400 0    50   Input ~ 0
 USB_UP_DN
-Text HLabel 5600 3000 0    50   Input ~ 0
+Text HLabel 7100 3200 2    50   Input ~ 0
 USB_DOWN1_DP
-Text HLabel 5600 3100 0    50   Input ~ 0
+Text HLabel 7100 3100 2    50   Input ~ 0
 USB_DOWN1_DN
-Text HLabel 5400 3400 0    50   Input ~ 0
+Text HLabel 7100 3500 2    50   Input ~ 0
 USB_DOWN2_DP
-Text HLabel 5400 3500 0    50   Input ~ 0
+Text HLabel 7100 3400 2    50   Input ~ 0
 USB_DOWN2_DN
+$Comp
+L chartreuse:USB2422 U?
+U 1 1 5CC65317
+P 6100 3700
+F 0 "U?" H 5500 4450 50  0000 C CNN
+F 1 "USB2422" H 5500 2950 50  0000 C CNN
+F 2 "" H 6100 3700 50  0001 C CNN
+F 3 "http://www.microchip.com/mymicrochip/filehandler.aspx?ddocname=en566992" H 6100 3700 50  0001 C CNN
+	1    6100 3700
+	1    0    0    -1
+$EndComp
+Wire Wire Line
+	5200 3400 5300 3400
+Wire Wire Line
+	5200 3500 5300 3500
+Wire Wire Line
+	7000 3400 7100 3400
+Wire Wire Line
+	7000 3500 7100 3500
+Wire Wire Line
+	7000 3100 7100 3100
+Wire Wire Line
+	7000 3200 7100 3200
+$Comp
+L power:GND #PWR?
+U 1 1 5CC68012
+P 6100 4700
+F 0 "#PWR?" H 6100 4450 50  0001 C CNN
+F 1 "GND" H 6105 4527 50  0000 C CNN
+F 2 "" H 6100 4700 50  0001 C CNN
+F 3 "" H 6100 4700 50  0001 C CNN
+	1    6100 4700
+	1    0    0    -1
+$EndComp
+Wire Wire Line
+	6100 4700 6100 4600
+$Comp
+L Device:C_Small C?
+U 1 1 5CC68116
+P 3250 4650
+F 0 "C?" H 3342 4696 50  0000 L CNN
+F 1 "C_Small" H 3342 4605 50  0000 L CNN
+F 2 "" H 3250 4650 50  0001 C CNN
+F 3 "~" H 3250 4650 50  0001 C CNN
+	1    3250 4650
+	1    0    0    -1
+$EndComp
+$Comp
+L Device:Ferrite_Bead_Small L?
+U 1 1 5CC68186
+P 4150 2700
+F 0 "L?" V 4005 2700 50  0000 C CNN
+F 1 "Ferrite_Bead_Small" V 4004 2700 50  0001 C CNN
+F 2 "" V 4080 2700 50  0001 C CNN
+F 3 "~" H 4150 2700 50  0001 C CNN
+	1    4150 2700
+	0    1    1    0
+$EndComp
+Wire Wire Line
+	6200 2700 6200 2800
+Wire Wire Line
+	6000 2800 6000 2700
+Connection ~ 6000 2700
+Wire Wire Line
+	6000 2700 6100 2700
+Wire Wire Line
+	6100 2800 6100 2700
+Connection ~ 6100 2700
+Wire Wire Line
+	6100 2700 6200 2700
+Wire Wire Line
+	5300 3100 5200 3100
+Wire Wire Line
+	5200 3100 5200 2700
+Connection ~ 5200 2700
+Wire Wire Line
+	5200 2700 6000 2700
+Wire Wire Line
+	5300 3200 5100 3200
+Wire Wire Line
+	5100 3200 5100 2700
+Wire Wire Line
+	4250 2700 5100 2700
+Connection ~ 5100 2700
+Wire Wire Line
+	5100 2700 5200 2700
 $EndSCHEMATC

Commit message: Finish USB circuit
Parts:
- added C?: 6pF, symbol Device:C_Small
- added C?: 1uF, symbol Device:C_Small
- added C?: 10uF, symbol Device:C_Small
- added C? (x3): 0.1uF, symbol Device:C_Small
- added R? (x4): 56K, symbol Device:R
- added Y?: 24M, symbol Device:Crystal_GND24_Small
- C?: value C_Small -> 6pF
- gave numbers to parts that had none: 1
Connections:
- net labels added: +3V3
- wire segments 19 -> 60
- no-connect marks 0 -> 5

Commit message: Change USB downstream port 1 to be non-removable
Connections:
- wire segments 60 -> 61

Commit message: Add component references
Parts:
- gave numbers to parts that had none: 13
Changed lines of the file:
@@
 encoding utf-8
 Sheet 3 4
-Title ""
-Date "2018-09-20"
-Rev ""
+Title "Chartreuse Main Board"
+Date "2018-09-21"
+Rev "0.9"
 Comp ""
 Comment1 ""
@@
 	6100 4900 6100 4600
 $Comp
-L Device:C_Small C?
+L Device:C_Small C206
 U 1 1 5CC68116
-P 3950 4650
-F 0 "C?" H 4042 4696 50  0000 L CNN
-F 1 "6pF" H 4042 4605 50  0000 L CNN
-F 2 "" H 3950 4650 50  0001 C CNN
-F 3 "~" H 3950 4650 50  0001 C CNN
-	1    3950 4650
-	1    0    0    -1
-$EndComp
-$Comp
-L Device:Ferrite_Bead_Small L?
+P 3850 4650
+F 0 "C206" H 3942 4696 50  0000 L CNN
+F 1 "6pF" H 3942 4605 50  0000 L CNN
+F 2 "" H 3850 4650 50  0001 C CNN
+F 3 "~" H 3850 4650 50  0001 C CNN
+	1    3850 4650
+	1    0    0    -1
+$EndComp
+$Comp
+L Device:Ferrite_Bead_Small FB2
 U 1 1 5CC68186
 P 3000 2700
-F 0 "L?" V 2855 2700 50  0000 C CNN
+F 0 "FB2" V 2855 2700 50  0000 C CNN
 F 1 "Ferrite_Bead_Small" V 2854 2700 50  0001 C CNN
 F 2 "" V 2930 2700 50  0001 C CNN
@@
 	5200 4300 5200 4500
 $Comp
-L Device:R R?
+L Device:R R203
 U 1 1 5BA46802
 P 5200 4650
-F 0 "R?" H 5270 4696 50  0000 L CNN
+F 0 "R203" H 5270 4696 50  0000 L CNN
 F 1 "56K" H 5270 4605 50  0000 L CNN
 F 2 "" V 5130 4650 50  0001 C CNN
@@
 $EndComp
 $Comp
-L Device:R R?
+L Device:R R202
 U 1 1 5BA4684F
-P 4900 4650
-F 0 "R?" H 4970 4696 50  0000 L CNN
-F 1 "56K" H 4970 4605 50  0000 L CNN
-F 2 "" V 4830 4650 50  0001 C CNN
-F 3 "~" H 4900 4650 50  0001 C CNN
-	1    4900 4650
-	1    0    0    -1
-$EndComp
-$Comp
-L Device:R R?
+P 4850 4650
+F 0 "R202" H 4920 4696 50  0000 L CNN
+F 1 "56K" H 4920 4605 50  0000 L CNN
+F 2 "" V 4780 4650 50  0001 C CNN
+F 3 "~" H 4850 4650 50  0001 C CNN
+	1    4850 4650
+	1    0    0    -1
+$EndComp
+$Comp
+L Device:R R201
 U 1 1 5BA468E7
 P 4800 2950
-F 0 "R?" H 4870 2996 50  0000 L CNN
+F 0 "R201" H 4870 2996 50  0000 L CNN
 F 1 "56K" H 4870 2905 50  0000 L CNN
 F 2 "" V 4730 2950 50  0001 C CNN
@@
 $EndComp
 Wire Wire Line
-	4900 4500 4900 4200
-Wire Wire Line
-	4900 4200 5300 4200
+	4850 4500 4850 4200
+Wire Wire Line
+	4850 4200 5300 4200
 Wire Wire Line
 	5300 4100 4800 4100
 $Comp
-L Device:C_Small C?
+L Device:C_Small C207
 U 1 1 5BA46F90
-P 4550 4650
-F 0 "C?" H 4642 4696 50  0000 L CNN
-F 1 "6pF" H 4642 4605 50  0000 L CNN
-F 2 "" H 4550 4650 50  0001 C CNN
-F 3 "~" H 4550 4650 50  0001 C CNN
-	1    4550 4650
-	1    0    0    -1
-$EndComp
-$Comp
-L Device:Crystal_GND24_Small Y?
+P 4450 4650
+F 0 "C207" H 4542 4696 50  0000 L CNN
+F 1 "6pF" H 4542 4605 50  0000 L CNN
+F 2 "" H 4450 4650 50  0001 C CNN
+F 3 "~" H 4450 4650 50  0001 C CNN
+	1    4450 4650
+	1    0    0    -1
+$EndComp
+$Comp
+L Device:Crystal_GND24_Small Y1
 U 1 1 5BA4707F
-P 4250 4400
-F 0 "Y?" H 4350 4450 50  0000 L CNN
-F 1 "24M" H 4350 4350 50  0000 L CNN
-F 2 "" H 4250 4400 50  0001 C CNN
-F 3 "~" H 4250 4400 50  0001 C CNN
-	1    4250 4400
-	1    0    0    -1
-$EndComp
-Wire Wire Line
-	4350 4400 4550 4400
-Wire Wire Line
-	4550 4400 4550 4550
-Wire Wire Line
-	4550 4400 4550 4000
-Wire Wire Line
-	4550 4000 5300 4000
-Connection ~ 4550 4400
-Wire Wire Line
-	5300 3900 3950 3900
-Wire Wire Line
-	3950 3900 3950 4400
-Wire Wire Line
-	3950 4400 4150 4400
-Wire Wire Line
-	3950 4550 3950 4400
-Connection ~ 3950 4400
+P 4150 4400
+F 0 "Y1" H 4250 4450 50  0000 L CNN
+F 1 "24M" H 4250 4350 50  0000 L CNN
+F 2 "" H 4150 4400 50  0001 C CNN
+F 3 "~" H 4150 4400 50  0001 C CNN
+	1    4150 4400
+	1    0    0    -1
+$EndComp
+Wire Wire Line
+	4250 4400 4450 4400
+Wire Wire Line
+	4450 4400 4450 4550
+Wire Wire Line
+	4450 4400 4450 4000
+Wire Wire Line
+	4450 4000 5300 4000
+Connection ~ 4450 4400
+Wire Wire Line
+	5300 3900 3850 3900
+Wire Wire Line
+	3850 3900 3850 4400
+Wire Wire Line
+	3850 4400 4050 4400
+Wire Wire Line
+	3850 4550 3850 4400
+Connection ~ 3850 4400
 $Comp
 L power:GND #PWR?
 U 1 1 5BA49008
-P 4250 4600
-F 0 "#PWR?" H 4250 4350 50  0001 C CNN
-F 1 "GND" H 4255 4427 50  0000 C CNN
-F 2 "" H 4250 4600 50  0001 C CNN
-F 3 "" H 4250 4600 50  0001 C CNN
-	1    4250 4600
-	1    0    0    -1
-$EndComp
-Wire Wire Line
-	4250 4525 4250 4600
-Wire Wire Line
-	4250 4200 4250 4275
+P 4150 4600
+F 0 "#PWR?" H 4150 4350 50  0001 C CNN
+F 1 "GND" H 4155 4427 50  0000 C CNN
+F 2 "" H 4150 4600 50  0001 C CNN
+F 3 "" H 4150 4600 50  0001 C CNN
+	1    4150 4600
+	1    0    0    -1
+$EndComp
+Wire Wire Line
+	4150 4525 4150 4600
+Wire Wire Line
+	4150 4200 4150 4275
 $Comp
 L power:GND #PWR?
 U 1 1 5BA4AC59
-P 4250 4200
-F 0 "#PWR?" H 4250 3950 50  0001 C CNN
-F 1 "GND" H 4255 4027 50  0000 C CNN
-F 2 "" H 4250 4200 50  0001 C CNN
-F 3 "" H 4250 4200 50  0001 C CNN
-	1    4250 4200
+P 4150 4200
+F 0 "#PWR?" H 4150 3950 50  0001 C CNN
+F 1 "GND" H 4155 4027 50  0000 C CNN
+F 2 "" H 4150 4200 50  0001 C CNN
+F 3 "" H 4150 4200 50  0001 C CNN
+	1    4150 4200
 	-1   0    0    1
 $EndComp
@@
 L power:GND #PWR?
 U 1 1 5BA4B6BA
-P 4550 4900
-F 0 "#PWR?" H 4550 4650 50  0001 C CNN
-F 1 "GND" H 4555 4727 50  0000 C CNN
-F 2 "" H 4550 4900 50  0001 C CNN
-F 3 "" H 4550 4900 50  0001 C CNN
-	1    4550 4900
+P 4450 4900
+F 0 "#PWR?" H 4450 4650 50  0001 C CNN
+F 1 "GND" H 4455 4727 50  0000 C CNN
+F 2 "" H 4450 4900 50  0001 C CNN
+F 3 "" H 4450 4900 50  0001 C CNN
+	1    4450 4900
 	1    0    0    -1
 $EndComp
@@
 L power:GND #PWR?
 U 1 1 5BA4B6EC
-P 3950 4900
-F 0 "#PWR?" H 3950 4650 50  0001 C CNN
-F 1 "GND" H 3955 4727 50  0000 C CNN
-F 2 "" H 3950 4900 50  0001 C CNN
-F 3 "" H 3950 4900 50  0001 C CNN
-	1    3950 4900
+P 3850 4900
+F 0 "#PWR?" H 3850 4650 50  0001 C CNN
+F 1 "GND" H 3855 4727 50  0000 C CNN
+F 2 "" H 3850 4900 50  0001 C CNN
+F 3 "" H 3850 4900 50  0001 C CNN
+	1    3850 4900
 	1    0    0    -1
 $EndComp
@@
 L power:GND #PWR?
 U 1 1 5BA4B71E
-P 4900 4900
-F 0 "#PWR?" H 4900 4650 50  0001 C CNN
-F 1 "GND" H 4905 4727 50  0000 C CNN
-F 2 "" H 4900 4900 50  0001 C CNN
-F 3 "" H 4900 4900 50  0001 C CNN
-	1    4900 4900
+P 4850 4900
+F 0 "#PWR?" H 4850 4650 50  0001 C CNN
+F 1 "GND" H 4855 4727 50  0000 C CNN
+F 2 "" H 4850 4900 50  0001 C CNN
+F 3 "" H 4850 4900 50  0001 C CNN
+	1    4850 4900
 	1    0    0    -1
 $EndComp
@@
 	5200 4900 5200 4800
 Wire Wire Line
-	3950 4750 3950 4900
-Wire Wire Line
-	4550 4750 4550 4900
-Wire Wire Line
-	4900 4800 4900 4900
-$Comp
-L Device:C_Small C?
+	3850 4750 3850 4900
+Wire Wire Line
+	4450 4750 4450 4900
+Wire Wire Line
+	4850 4800 4850 4900
+$Comp
+L Device:C_Small C205
 U 1 1 5BA4DC88
-P 3550 4650
-F 0 "C?" H 3642 4696 50  0000 L CNN
-F 1 "1uF" H 3642 4605 50  0000 L CNN
-F 2 "" H 3550 4650 50  0001 C CNN
-F 3 "~" H 3550 4650 50  0001 C CNN
-	1    3550 4650
+P 3450 4650
+F 0 "C205" H 3542 4696 50  0000 L CNN
+F 1 "1uF" H 3542 4605 50  0000 L CNN
+F 2 "" H 3450 4650 50  0001 C CNN
+F 3 "~" H 3450 4650 50  0001 C CNN
+	1    3450 4650
 	1    0    0    -1
 $EndComp
@@
 L power:GND #PWR?
 U 1 1 5BA4DCEA
-P 3550 4900
-F 0 "#PWR?" H 3550 4650 50  0001 C CNN
-F 1 "GND" H 3555 4727 50  0000 C CNN
-F 2 "" H 3550 4900 50  0001 C CNN
-F 3 "" H 3550 4900 50  0001 C CNN
-	1    3550 4900
-	1    0    0    -1
-$EndComp
-Wire Wire Line
-	3550 4750 3550 4900
-Wire Wire Line
-	3550 4550 3550 3800
-Wire Wire Line
-	3550 3800 5300 3800
-$Comp
-L Device:R R?
+P 3450 4900
+F 0 "#PWR?" H 3450 4650 50  0001 C CNN
+F 1 "GND" H 3455 4727 50  0000 C CNN
+F 2 "" H 3450 4900 50  0001 C CNN
+F 3 "" H 3450 4900 50  0001 C CNN
+	1    3450 4900
+	1    0    0    -1
+$EndComp
+Wire Wire Line
+	3450 4750 3450 4900
+Wire Wire Line
+	3450 4550 3450 3800
+Wire Wire Line
+	3450 3800 5300 3800
+$Comp
+L Device:R R204
 U 1 1 5BA50317
 P 7100 4650
-F 0 "R?" H 7170 4696 50  0000 L CNN
+F 0 "R204" H 7170 4696 50  0000 L CNN
 F 1 "56K" H 7170 4605 50  0000 L CNN
 F 2 "" V 7030 4650 50  0001 C CNN
@@
 NoConn ~ 7000 3700
 $Comp
-L Device:C_Small C?
+L Device:C_Small C204
 U 1 1 5BA558FB
 P 4400 2900
-F 0 "C?" H 4492 2946 50  0000 L CNN
+F 0 "C204" H 4492 2946 50  0000 L CNN
 F 1 "10uF" H 4492 2855 50  0000 L CNN
 F 2 "" H 4400 2900 50  0001 C CNN
@@
 	4400 2700 4800 2700
 $Comp
-L Device:C_Small C?
+L Device:C_Small C203
 U 1 1 5BA593DA
 P 4000 2900
-F 0 "C?" H 4092 2946 50  0000 L CNN
+F 0 "C203" H 4092 2946 50  0000 L CNN
 F 1 "0.1uF" H 4092 2855 50  0000 L CNN
 F 2 "" H 4000 2900 50  0001 C CNN
@@
 	4000 3000 4000 3100
 $Comp
-L Device:C_Small C?
+L Device:C_Small C202
 U 1 1 5BA5A04D
 P 3600 2900
-F 0 "C?" H 3692 2946 50  0000 L CNN
+F 0 "C202" H 3692 2946 50  0000 L CNN
 F 1 "0.1uF" H 3692 2855 50  0000 L CNN
 F 2 "" H 3600 2900 50  0001 C CNN
@@
 	3600 3000 3600 3100
 $Comp
-L Device:C_Small C?
+L Device:C_Small C201
 U 1 1 5BA5A05A
 P 3200 2900
-F 0 "C?" H 3292 2946 50  0000 L CNN
+F 0 "C201" H 3292 2946 50  0000 L CNN
 F 1 "0.1uF" H 3292 2855 50  0000 L CNN
 F 2 "" H 3200 2900 50  0001 C CNN

Commit message: Preliminary assign footprints
Parts:
- C201, C202, C203, C205, C206, C207: footprint (none) -> Capacitors_SMD:C_0402
- C204: footprint (none) -> Capacitors_SMD:C_0805
- FB2: footprint (none) -> Resistors_SMD:R_0603
- R201, R202, R203, R204: footprint (none) -> Resistors_SMD:R_0402
- U8: footprint (none) -> Housings_DFN_QFN:QFN-24-1EP_4x4mm_Pitch0.5mm
- Y1: footprint (none) -> Crystals:Crystal_SMD_0603-4pin_6.0x3.5mm
Changed lines of the file:
@@
 F 0 "U8" H 5500 4450 50  0000 C CNN
 F 1 "USB2422" H 5500 2950 50  0000 C CNN
-F 2 "" H 6100 3700 50  0001 C CNN
+F 2 "Housings_DFN_QFN:QFN-24-1EP_4x4mm_Pitch0.5mm" H 6100 3700 50  0001 C CNN
 F 3 "http://www.microchip.com/mymicrochip/filehandler.aspx?ddocname=en566992" H 6100 3700 50  0001 C CNN
 	1    6100 3700
@@
 F 0 "C206" H 3942 4696 50  0000 L CNN
 F 1 "6pF" H 3942 4605 50  0000 L CNN
-F 2 "" H 3850 4650 50  0001 C CNN
+F 2 "Capacitors_SMD:C_0402" H 3850 4650 50  0001 C CNN
 F 3 "~" H 3850 4650 50  0001 C CNN
 	1    3850 4650
@@
 F 0 "FB2" V 2855 2700 50  0000 C CNN
 F 1 "Ferrite_Bead_Small" V 2854 2700 50  0001 C CNN
-F 2 "" V 2930 2700 50  0001 C CNN
+F 2 "Resistors_SMD:R_0603" V 2930 2700 50  0001 C CNN
 F 3 "~" H 3000 2700 50  0001 C CNN
 	1    3000 2700
@@
 F 0 "R203" H 5270 4696 50  0000 L CNN
 F 1 "56K" H 5270 4605 50  0000 L CNN
-F 2 "" V 5130 4650 50  0001 C CNN
+F 2 "Resistors_SMD:R_0402" V 5130 4650 50  0001 C CNN
 F 3 "~" H 5200 4650 50  0001 C CNN
 	1    5200 4650
@@
 F 0 "R202" H 4920 4696 50  0000 L CNN
 F 1 "56K" H 4920 4605 50  0000 L CNN
-F 2 "" V 4780 4650 50  0001 C CNN
+F 2 "Resistors_SMD:R_0402" V 4780 4650 50  0001 C CNN
 F 3 "~" H 4850 4650 50  0001 C CNN
 	1    4850 4650
@@
 F 0 "R201" H 4870 2996 50  0000 L CNN
 F 1 "56K" H 4870 2905 50  0000 L CNN
-F 2 "" V 4730 2950 50  0001 C CNN
+F 2 "Resistors_SMD:R_0402" V 4730 2950 50  0001 C CNN
 F 3 "~" H 4800 2950 50  0001 C CNN
 	1    4800 2950
@@
 F 0 "C207" H 4542 4696 50  0000 L CNN
 F 1 "6pF" H 4542 4605 50  0000 L CNN
-F 2 "" H 4450 4650 50  0001 C CNN
+F 2 "Capacitors_SMD:C_0402" H 4450 4650 50  0001 C CNN
 F 3 "~" H 4450 4650 50  0001 C CNN
 	1    4450 4650
@@
 F 0 "Y1" H 4250 4450 50  0000 L CNN
 F 1 "24M" H 4250 4350 50  0000 L CNN
-F 2 "" H 4150 4400 50  0001 C CNN
+F 2 "Crystals:Crystal_SMD_0603-4pin_6.0x3.5mm" H 4150 4400 50  0001 C CNN
 F 3 "~" H 4150 4400 50  0001 C CNN
 	1    4150 4400
@@
 F 0 "C205" H 3542 4696 50  0000 L CNN
 F 1 "1uF" H 3542 4605 50  0000 L CNN
-F 2 "" H 3450 4650 50  0001 C CNN
+F 2 "Capacitors_SMD:C_0402" H 3450 4650 50  0001 C CNN
 F 3 "~" H 3450 4650 50  0001 C CNN
 	1    3450 4650
@@
 F 0 "R204" H 7170 4696 50  0000 L CNN
 F 1 "56K" H 7170 4605 50  0000 L CNN
-F 2 "" V 7030 4650 50  0001 C CNN
+F 2 "Resistors_SMD:R_0402" V 7030 4650 50  0001 C CNN
 F 3 "~" H 7100 4650 50  0001 C CNN
 	1    7100 4650
@@
 F 0 "C204" H 4492 2946 50  0000 L CNN
 F 1 "10uF" H 4492 2855 50  0000 L CNN
-F 2 "" H 4400 2900 50  0001 C CNN
+F 2 "Capacitors_SMD:C_0805" H 4400 2900 50  0001 C CNN
 F 3 "~" H 4400 2900 50  0001 C CNN
 	1    4400 2900
@@
 F 0 "C203" H 4092 2946 50  0000 L CNN
 F 1 "0.1uF" H 4092 2855 50  0000 L CNN
-F 2 "" H 4000 2900 50  0001 C CNN
+F 2 "Capacitors_SMD:C_0402" H 4000 2900 50  0001 C CNN
 F 3 "~" H 4000 2900 50  0001 C CNN
 	1    4000 2900
@@
 F 0 "C202" H 3692 2946 50  0000 L CNN
 F 1 "0.1uF" H 3692 2855 50  0000 L CNN
-F 2 "" H 3600 2900 50  0001 C CNN
+F 2 "Capacitors_SMD:C_0402" H 3600 2900 50  0001 C CNN
 F 3 "~" H 3600 2900 50  0001 C CNN
 	1    3600 2900
@@
 F 0 "C201" H 3292 2946 50  0000 L CNN
 F 1 "0.1uF" H 3292 2855 50  0000 L CNN
-F 2 "" H 3200 2900 50  0001 C CNN
+F 2 "Capacitors_SMD:C_0402" H 3200 2900 50  0001 C CNN
 F 3 "~" H 3200 2900 50  0001 C CNN
 	1    3200 2900

Commit message: Revise component numbering and footprints
Parts:
- FB2: value Ferrite_Bead_Small -> BLM18RK601SN1D
Changed lines of the file:
@@
 P 3000 2700
 F 0 "FB2" V 2855 2700 50  0000 C CNN
-F 1 "Ferrite_Bead_Small" V 2854 2700 50  0001 C CNN
+F 1 "BLM18RK601SN1D" V 2854 2700 50  0001 C CNN
 F 2 "Resistors_SMD:R_0603" V 2930 2700 50  0001 C CNN
 F 3 "~" H 3000 2700 50  0001 C CNN
