File: hardware/mainboard/chartreuse/chartreuse.sch (KiCad schematic (older format))
At the start: 0 parts

Commit message: Add power supply schematic sheet
Added a hierarchical sheet for power circuit and TPS61090 boost converter.
Parts:
- added BT1: LiPo, symbol Device:Battery_Cell
- added J1: USB_B_Micro, symbol Connector:USB_B_Micro
- added J2: USB_A, symbol Connector:USB_A
- added U3: LM1117-3.3, symbol Regulator_Linear:LM1117-3.3
Connections:
- net labels added: GND, VBUS
- wire segments 0 -> 13
- no-connect marks 0 -> 3
Other:
- note added: "Charger Input"
Changed lines of the file:
@@
 $Descr A 11000 8500
 encoding utf-8
-Sheet 1 1
+Sheet 1 2
 Title "Chartreuse Main Board"
 Date "2018-06-10"
@@
 Comment4 ""
 $EndDescr
+$Comp
+L Connector:USB_B_Micro J1
+U 1 1 5B1DED94
+P 900 1300
+F 0 "J1" H 955 1767 50  0000 C CNN
+F 1 "USB_B_Micro" H 955 1676 50  0000 C CNN
+F 2 "" H 1050 1250 50  0001 C CNN
+F 3 "~" H 1050 1250 50  0001 C CNN
+	1    900  1300
+	1    0    0    -1
+$EndComp
+$Comp
+L Connector:USB_A J2
+U 1 1 5B1DEE2E
+P 4850 1200
+F 0 "J2" H 4620 1191 50  0000 R CNN
+F 1 "USB_A" H 4620 1100 50  0000 R CNN
+F 2 "" H 5000 1150 50  0001 C CNN
+F 3 " ~" H 5000 1150 50  0001 C CNN
+	1    4850 1200
+	-1   0    0    -1
+$EndComp
+$Comp
+L power:GND #PWR0101
+U 1 1 5B1DEF29
+P 800 1800
+F 0 "#PWR0101" H 800 1550 50  0001 C CNN
+F 1 "GND" H 805 1627 50  0000 C CNN
+F 2 "" H 800 1800 50  0001 C CNN
+F 3 "" H 800 1800 50  0001 C CNN
+	1    800  1800
+	1    0    0    -1
+$EndComp
+Wire Wire Line
+	800  1800 800  1700
+$Comp
+L power:GND #PWR0102
+U 1 1 5B1DEF80
+P 900 1800
+F 0 "#PWR0102" H 900 1550 50  0001 C CNN
+F 1 "GND" H 905 1627 50  0000 C CNN
+F 2 "" H 900 1800 50  0001 C CNN
+F 3 "" H 900 1800 50  0001 C CNN
+	1    900  1800
+	1    0    0    -1
+$EndComp
+NoConn ~ 1200 1500
+NoConn ~ 1200 1400
+NoConn ~ 1200 1300
+$Comp
+L Regulator_Linear:LM1117-3.3 U3
+U 1 1 5B1DF129
+P 3250 1300
+F 0 "U3" H 3250 1542 50  0000 C CNN
+F 1 "LM1117-3.3" H 3250 1451 50  0000 C CNN
+F 2 "" H 3250 1300 50  0001 C CNN
+F 3 "http://www.ti.com/lit/ds/symlink/lm1117.pdf" H 3250 1300 50  0001 C CNN
+	1    3250 1300
+	1    0    0    -1
+$EndComp
+$Comp
+L Device:Battery_Cell BT1
+U 1 1 5B1DF1E1
+P 1700 1500
+F 0 "BT1" H 1818 1596 50  0000 L CNN
+F 1 "LiPo" H 1818 1505 50  0000 L CNN
+F 2 "" V 1700 1560 50  0001 C CNN
+F 3 "~" V 1700 1560 50  0001 C CNN
+	1    1700 1500
+	-1   0    0    -1
+$EndComp
+$Sheet
+S 1900 1000 550  400
+U 5B1DF219
+F0 "Power Supply" 50
+F1 "chartreuse-power.sch" 50
+F2 "VCHARGE" I L 1900 1100 50
+F3 "VLIPO" I L 1900 1200 50
+F4 "VBUS" I R 2450 1300 50
+$EndSheet
+Wire Wire Line
+	1900 1100 1200 1100
+Wire Wire Line
+	1700 1300 1700 1200
+Wire Wire Line
+	1700 1200 1900 1200
+Wire Wire Line
+	1700 1600 1700 1700
+$Comp
+L power:GND #PWR0103
+U 1 1 5B1DF78F
+P 1700 1700
+F 0 "#PWR0103" H 1700 1450 50  0001 C CNN
+F 1 "GND" H 1705 1527 50  0000 C CNN
+F 2 "" H 1700 1700 50  0001 C CNN
+F 3 "" H 1700 1700 50  0001 C CNN
+	1    1700 1700
+	1    0    0    -1
+$EndComp
+Wire Wire Line
+	900  1700 900  1800
+Wire Wire Line
+	2950 1300 2850 1300
+$Comp
+L power:GND #PWR0104
+U 1 1 5B1DFB61
+P 3250 1700
+F 0 "#PWR0104" H 3250 1450 50  0001 C CNN
+F 1 "GND" H 3255 1527 50  0000 C CNN
+F 2 "" H 3250 1700 50  0001 C CNN
+F 3 "" H 3250 1700 50  0001 C CNN
+	1    3250 1700
+	1    0    0    -1
+$EndComp
+Wire Wire Line
+	3250 1700 3250 1600
+$Comp
+L power:VBUS #PWR0105
+U 1 1 5B1DFBEF
+P 2850 1200
+F 0 "#PWR0105" H 2850 1050 50  0001 C CNN
+F 1 "VBUS" H 2865 1373 50  0000 C CNN
+F 2 "" H 2850 1200 50  0001 C CNN
+F 3 "" H 2850 1200 50  0001 C CNN
+	1    2850 1200
+	1    0    0    -1
+$EndComp
+Wire Wire Line
+	2850 1200 2850 1300
+Connection ~ 2850 1300
+Wire Wire Line
+	2850 1300 2450 1300
+$Comp
+L power:VBUS #PWR0106
+U 1 1 5B1DFC6E
+P 4450 1000
+F 0 "#PWR0106" H 4450 850 50  0001 C CNN
+F 1 "VBUS" V 4465 1127 50  0000 L CNN
+F 2 "" H 4450 1000 50  0001 C CNN
+F 3 "" H 4450 1000 50  0001 C CNN
+	1    4450 1000
+	0    -1   -1   0
+$EndComp
+Wire Wire Line
+	4550 1000 4450 1000
+$Comp
+L power:GND #PWR0107
+U 1 1 5B1DFDCA
+P 4850 1700
+F 0 "#PWR0107" H 4850 1450 50  0001 C CNN
+F 1 "GND" H 4855 1527 50  0000 C CNN
+F 2 "" H 4850 1700 50  0001 C CNN
+F 3 "" H 4850 1700 50  0001 C CNN
+	1    4850 1700
+	1    0    0    -1
+$EndComp
+$Comp
+L power:GND #PWR0108
+U 1 1 5B1DFDF4
+P 4950 1700
+F 0 "#PWR0108" H 4950 1450 50  0001 C CNN
+F 1 "GND" H 4955 1527 50  0000 C CNN
+F 2 "" H 4950 1700 50  0001 C CNN
+F 3 "" H 4950 1700 50  0001 C CNN
+	1    4950 1700
+	1    0    0    -1
+$EndComp
+Wire Wire Line
+	4950 1700 4950 1600
+Wire Wire Line
+	4850 1700 4850 1600
+Text Notes 700  750  0    50   ~ 0
+Charger Input
 $EndSCHEMATC

Commit message: Add project-specific component library
Create components for TFP401, AR1100, 24LC02, USB2422, and FAN5333. In addition, add schematic sheets for HDMI and USB subsections.
Parts:
- added FB1: Ferrite, symbol Device:Ferrite_Bead_Small
- added J2: USB_B_Micro, symbol Connector:USB_B_Micro
- renumbered J2 to J3
Connections:
- net labels added: +3V3, +5V
- wire segments 13 -> 32
- no-connect marks 3 -> 4
Other:
- note added: "Female USB-A\nFlash Drive"
- note added: "Raspberry Pi"
- moved on the sheet: U3

Commit message: Finish HDMI circuit (mostly)
Added most of the connections and minor components in the HDMI sheet. In addition, added the USB hub IC to the USB sheet.
Parts:
- added C? (x2): 10uF, symbol Device:C_Small
Connections:
- wire segments 32 -> 36
Other:
- moved on the sheet: U3

Commit message: Add component references
Parts:
- gave numbers to parts that had none: 2
Other:
- moved on the sheet: U3
Changed lines of the file:
@@
 Sheet 1 4
 Title "Chartreuse Main Board"
-Date "2018-06-10"
+Date "2018-09-21"
 Rev "0.9"
 Comp ""
@@
 L Regulator_Linear:LM1117-3.3 U3
 U 1 1 5B1DF129
-P 6300 2100
-F 0 "U3" H 6300 2342 50  0000 C CNN
-F 1 "LM1117-3.3" H 6300 2251 50  0000 C CNN
-F 2 "" H 6300 2100 50  0001 C CNN
-F 3 "http://www.ti.com/lit/ds/symlink/lm1117.pdf" H 6300 2100 50  0001 C CNN
-	1    6300 2100
+P 6350 2100
+F 0 "U3" H 6350 2342 50  0000 C CNN
+F 1 "LM1117-3.3" H 6350 2251 50  0000 C CNN
+F 2 "" H 6350 2100 50  0001 C CNN
+F 3 "http://www.ti.com/lit/ds/symlink/lm1117.pdf" H 6350 2100 50  0001 C CNN
+	1    6350 2100
 	1    0    0    -1
 $EndComp
@@
 L power:GND #PWR0104
 U 1 1 5B1DFB61
-P 6300 2500
-F 0 "#PWR0104" H 6300 2250 50  0001 C CNN
-F 1 "GND" H 6305 2327 50  0000 C CNN
-F 2 "" H 6300 2500 50  0001 C CNN
-F 3 "" H 6300 2500 50  0001 C CNN
-	1    6300 2500
-	1    0    0    -1
-$EndComp
-Wire Wire Line
-	6300 2500 6300 2400
+P 6350 2500
+F 0 "#PWR0104" H 6350 2250 50  0001 C CNN
+F 1 "GND" H 6355 2327 50  0000 C CNN
+F 2 "" H 6350 2500 50  0001 C CNN
+F 3 "" H 6350 2500 50  0001 C CNN
+	1    6350 2500
+	1    0    0    -1
+$EndComp
+Wire Wire Line
+	6350 2500 6350 2400
 $Comp
 L power:VBUS #PWR0106
@@
 L power:+3V3 #PWR0105
 U 1 1 5B21CB65
-P 6700 1900
-F 0 "#PWR0105" H 6700 1750 50  0001 C CNN
-F 1 "+3V3" H 6715 2073 50  0000 C CNN
-F 2 "" H 6700 1900 50  0001 C CNN
-F 3 "" H 6700 1900 50  0001 C CNN
-	1    6700 1900
+P 6750 1900
+F 0 "#PWR0105" H 6750 1750 50  0001 C CNN
+F 1 "+3V3" H 6765 2073 50  0000 C CNN
+F 2 "" H 6750 1900 50  0001 C CNN
+F 3 "" H 6750 1900 50  0001 C CNN
+	1    6750 1900
 	1    0    0    -1
 $EndComp
@@
 $EndSheet
 Wire Wire Line
-	6600 2100 6700 2100
-Wire Wire Line
-	6700 2100 6700 1900
+	6650 2100 6750 2100
+Wire Wire Line
+	6750 2100 6750 1900
 $Sheet
 S 4600 4050 1000 800
@@
 	3300 2550 3300 2500
 $Comp
-L Device:C_Small C?
+L Device:C_Small C401
 U 1 1 5BA58A78
 P 5800 2300
-F 0 "C?" H 5892 2346 50  0000 L CNN
+F 0 "C401" H 5892 2346 50  0000 L CNN
 F 1 "10uF" H 5892 2255 50  0000 L CNN
 F 2 "" H 5800 2300 50  0001 C CNN
@@
 	5800 2500 5800 2400
 $Comp
-L Device:C_Small C?
+L Device:C_Small C402
 U 1 1 5BA594E5
-P 6700 2300
-F 0 "C?" H 6792 2346 50  0000 L CNN
-F 1 "10uF" H 6792 2255 50  0000 L CNN
-F 2 "" H 6700 2300 50  0001 C CNN
-F 3 "~" H 6700 2300 50  0001 C CNN
-	1    6700 2300
+P 6750 2300
+F 0 "C402" H 6842 2346 50  0000 L CNN
+F 1 "10uF" H 6842 2255 50  0000 L CNN
+F 2 "" H 6750 2300 50  0001 C CNN
+F 3 "~" H 6750 2300 50  0001 C CNN
+	1    6750 2300
 	1    0    0    -1
 $EndComp
@@
 L power:GND #PWR?
 U 1 1 5BA594EB
-P 6700 2500
-F 0 "#PWR?" H 6700 2250 50  0001 C CNN
-F 1 "GND" H 6705 2327 50  0000 C CNN
-F 2 "" H 6700 2500 50  0001 C CNN
-F 3 "" H 6700 2500 50  0001 C CNN
-	1    6700 2500
-	1    0    0    -1
-$EndComp
-Wire Wire Line
-	6700 2500 6700 2400
-Wire Wire Line
-	6700 2200 6700 2100
-Connection ~ 6700 2100
+P 6750 2500
+F 0 "#PWR?" H 6750 2250 50  0001 C CNN
+F 1 "GND" H 6755 2327 50  0000 C CNN
+F 2 "" H 6750 2500 50  0001 C CNN
+F 3 "" H 6750 2500 50  0001 C CNN
+	1    6750 2500
+	1    0    0    -1
+$EndComp
+Wire Wire Line
+	6750 2500 6750 2400
+Wire Wire Line
+	6750 2200 6750 2100
+Connection ~ 6750 2100
 Wire Wire Line
 	5150 2100 5800 2100
@@
 Connection ~ 5800 2100
 Wire Wire Line
-	5800 2100 6000 2100
+	5800 2100 6050 2100
 Wire Wire Line
 	5800 2100 5800 2200

Commit message: Schematic DRC check
Connections:
- net labels removed: VBUS
Changed lines of the file:
@@
 Wire Wire Line
 	6350 2500 6350 2400
-$Comp
-L power:VBUS #PWR0106
-U 1 1 5B1DFC6E
-P 6250 5050
-F 0 "#PWR0106" H 6250 4900 50  0001 C CNN
-F 1 "VBUS" V 6265 5177 50  0000 L CNN
-F 2 "" H 6250 5050 50  0001 C CNN
-F 3 "" H 6250 5050 50  0001 C CNN
-	1    6250 5050
-	0    -1   -1   0
-$EndComp
 Wire Wire Line
 	6350 5050 6250 5050
@@
 $EndComp
 $Comp
-L power:GND #PWR?
+L power:GND #PWR0128
 U 1 1 5BA58AEA
 P 5800 2500
-F 0 "#PWR?" H 5800 2250 50  0001 C CNN
+F 0 "#PWR0128" H 5800 2250 50  0001 C CNN
 F 1 "GND" H 5805 2327 50  0000 C CNN
 F 2 "" H 5800 2500 50  0001 C CNN
@@
 $EndComp
 $Comp
-L power:GND #PWR?
+L power:GND #PWR0129
 U 1 1 5BA594EB
 P 6750 2500
-F 0 "#PWR?" H 6750 2250 50  0001 C CNN
+F 0 "#PWR0129" H 6750 2250 50  0001 C CNN
 F 1 "GND" H 6755 2327 50  0000 C CNN
 F 2 "" H 6750 2500 50  0001 C CNN
@@
 Wire Wire Line
 	5800 2100 5800 2200
+$Comp
+L power:+5V #PWR0106
+U 1 1 5BABD433
+P 6250 5050
+F 0 "#PWR0106" H 6250 4900 50  0001 C CNN
+F 1 "+5V" V 6265 5178 50  0000 L CNN
+F 2 "" H 6250 5050 50  0001 C CNN
+F 3 "" H 6250 5050 50  0001 C CNN
+	1    6250 5050
+	0    -1   -1   0
+$EndComp
 $EndSCHEMATC

Commit message: Preliminary assign footprints
Parts:
- BT1: footprint (none) -> Connectors_JST:JST_PH_S2B-PH-SM4-TB_02x2.00mm_Angled
- C401, C402: footprint (none) -> Capacitors_SMD:CP_Elec_4x5.8
- FB1: footprint (none) -> Resistors_SMD:R_0603
- J1: footprint (none) -> Connectors_USB:USB_Micro-B_Molex_47346-0001
- J2: footprint (none) -> SMD_Packages:Conn-5
- U3: footprint (none) -> TO_SOT_Packages_SMD:SOT-223-3_TabPin2
Changed lines of the file:
@@
 F 0 "J1" H 3455 2567 50  0000 C CNN
 F 1 "USB_B_Micro" H 3455 2476 50  0000 C CNN
-F 2 "" H 3550 2050 50  0001 C CNN
+F 2 "Connectors_USB:USB_Micro-B_Molex_47346-0001" H 3550 2050 50  0001 C CNN
 F 3 "~" H 3550 2050 50  0001 C CNN
 	1    3400 2100
@@
 F 0 "U3" H 6350 2342 50  0000 C CNN
 F 1 "LM1117-3.3" H 6350 2251 50  0000 C CNN
-F 2 "" H 6350 2100 50  0001 C CNN
+F 2 "TO_SOT_Packages_SMD:SOT-223-3_TabPin2" H 6350 2100 50  0001 C CNN
 F 3 "http://www.ti.com/lit/ds/symlink/lm1117.pdf" H 6350 2100 50  0001 C CNN
 	1    6350 2100
@@
 F 0 "BT1" H 4518 2396 50  0000 L CNN
 F 1 "LiPo" H 4518 2305 50  0000 L CNN
-F 2 "" V 4400 2360 50  0001 C CNN
+F 2 "Connectors_JST:JST_PH_S2B-PH-SM4-TB_02x2.00mm_Angled" V 4400 2360 50  0001 C CNN
 F 3 "~" V 4400 2360 50  0001 C CNN
 	1    4400 2300
@@
 F 0 "J2" H 4155 4617 50  0000 C CNN
 F 1 "USB_B_Micro" H 4155 4526 50  0000 C CNN
-F 2 "" H 4250 4100 50  0001 C CNN
+F 2 "SMD_Packages:Conn-5" H 4250 4100 50  0001 C CNN
 F 3 "~" H 4250 4100 50  0001 C CNN
 	1    4100 4150
@@
 F 0 "FB1" H 3100 2746 50  0000 L CNN
 F 1 "Ferrite" H 3100 2655 50  0000 L CNN
-F 2 "" V 2930 2700 50  0001 C CNN
+F 2 "Resistors_SMD:R_0603" V 2930 2700 50  0001 C CNN
 F 3 "~" H 3000 2700 50  0001 C CNN
 	1    3000 2700
@@
 F 0 "C401" H 5892 2346 50  0000 L CNN
 F 1 "10uF" H 5892 2255 50  0000 L CNN
-F 2 "" H 5800 2300 50  0001 C CNN
+F 2 "Capacitors_SMD:CP_Elec_4x5.8" H 5800 2300 50  0001 C CNN
 F 3 "~" H 5800 2300 50  0001 C CNN
 	1    5800 2300
@@
 F 0 "C402" H 6842 2346 50  0000 L CNN
 F 1 "10uF" H 6842 2255 50  0000 L CNN
-F 2 "" H 6750 2300 50  0001 C CNN
+F 2 "Capacitors_SMD:CP_Elec_4x5.8" H 6750 2300 50  0001 C CNN
 F 3 "~" H 6750 2300 50  0001 C CNN
 	1    6750 2300

Commit message: Revise component numbering and footprints
Parts:
- FB1: value Ferrite -> BLM18RK601SN1D
- renumbered BT1 to J3, J3 to J4
Changed lines of the file:
@@
 $EndComp
 $Comp
-L Connector:USB_A J3
+L Connector:USB_A J4
 U 1 1 5B1DEE2E
 P 6650 5250
-F 0 "J3" H 6420 5241 50  0000 R CNN
+F 0 "J4" H 6420 5241 50  0000 R CNN
 F 1 "USB_A" H 6420 5150 50  0000 R CNN
 F 2 "" H 6800 5200 50  0001 C CNN
@@
 $EndComp
 $Comp
-L Device:Battery_Cell BT1
+L Device:Battery_Cell J3
 U 1 1 5B1DF1E1
 P 4400 2300
-F 0 "BT1" H 4518 2396 50  0000 L CNN
+F 0 "J3" H 4518 2396 50  0000 L CNN
 F 1 "LiPo" H 4518 2305 50  0000 L CNN
 F 2 "Connectors_JST:JST_PH_S2B-PH-SM4-TB_02x2.00mm_Angled" V 4400 2360 50  0001 C CNN
@@
 P 3000 2700
 F 0 "FB1" H 3100 2746 50  0000 L CNN
-F 1 "Ferrite" H 3100 2655 50  0000 L CNN
+F 1 "BLM18RK601SN1D" H 3100 2655 50  0001 L CNN
 F 2 "Resistors_SMD:R_0603" V 2930 2700 50  0001 C CNN
 F 3 "~" H 3000 2700 50  0001 C CNN
