File: hardware/mainboard/chartreuse/chartreuse.sch (KiCad schematic (older format))
At the start: 8 parts, among them J1 USB_B_Micro, J2 USB_B_Micro, J3 LiPo, J4 USB_A, U3 LM1117-3.3

Commit message: Add netlist to PCB design
Parts:
- J4: footprint (none) -> Connectors:USB_A
Changed lines of the file:
@@
 F 0 "J4" H 6420 5241 50  0000 R CNN
 F 1 "USB_A" H 6420 5150 50  0000 R CNN
-F 2 "" H 6800 5200 50  0001 C CNN
+F 2 "Connectors:USB_A" H 6800 5200 50  0001 C CNN
 F 3 " ~" H 6800 5200 50  0001 C CNN
 	1    6650 5250
