File: hardware/mainboard/chartreuse/chartreuse-hdmi.sch (KiCad schematic (older format))
At the start: 13 parts, among them J6 FFC-40

Commit message: Add to HDMI circuit U4, U5, U6, U7, and U8
Parts:
- added C? (x4): 0.1uF, symbol Device:C_Small
- added C? (x2): 12pF, symbol Device:C_Small
- added C? (x2): 1uF, symbol Device:C_Small
- added C?: 10uF, symbol Device:C_Small
- added D?: MBR0540, symbol Device:D
- added D?: MM3Z24VT1G, symbol Device:D
- added D?: 1N4148, symbol Device:D_Small
- added J5: FFC-20, symbol Connector_Generic:Conn_01x20
- added L?: Ferrite_Bead_Small, symbol Device:Ferrite_Bead_Small
- added L?: BRL3225T150K, symbol Device:L
- added LED1: RED, symbol Device:LED
- added LED3: BLUE, symbol Device:LED
- added Q?: BSS138, Package_TO_SOT_SMD:SOT-23, symbol Transistor_FET:BSS138
- added R?: 10K, symbol Device:R
- added R?: R, symbol Device:R
- added R?: 1K, symbol Device:R
- added R?: 3, symbol Device:R
- added R? (x2): 12, symbol Device:R
- added R? (x4): 10K, symbol Device:R_Small
- added U5: 24LC02BT-OT, symbol chartreuse:24LC02BT-OT
- added Y?: 12M, symbol Device:Crystal_Small
- gave numbers to parts that had none: 3
Connections:
- net labels added: +24V, HDMI_5V, HDMI_DDC_CLK, HDMI_DDC_DTA, HDMI_HOTPLUG, HDMI_TMDS0_N, HDMI_TMDS0_P, HDMI_TMDS1_N, HDMI_TMDS1_P, HDMI_TMDS2_N, HDMI_TMDS2_P, HDMI_TMDSC_N, HDMI_TMDSC_P, VBUS
- wire segments 120 -> 281
- no-connect marks 29 -> 32
Other:
- moved on the sheet: U4

Commit message: Finish HDMI circuit (mostly)
Added most of the connections and minor components in the HDMI sheet. In addition, added the USB hub IC to the USB sheet.
Parts:
- added C? (x6): 10uF, symbol Device:C_Small
- added C? (x13): 0.1uF, symbol Device:C_Small
- added L?: BLM18RK601SN1D, symbol Device:Ferrite_Bead_Small
- added L? (x4): Ferrite_Bead_Small, symbol Device:Ferrite_Bead_Small
- R?: value R -> 1K
Connections:
- net labels added: +3V3, +5V
- net labels removed: VBUS, VDD
- wire segments 281 -> 381
- no-connect marks 32 -> 34
Other:
- moved on the sheet: U4

Commit message: Add component references
Parts:
- gave numbers to parts that had none: 58
- renumbered LED1 to D2, LED3 to D3

Commit message: Schematic DRC check
Parts:
- renumbered C318 to C332
Connections:
- net labels removed: +24V
- wire segments 381 -> 382

Commit message: Preliminary assign footprints
Parts:
- C301, C302, C303, C304, C326, C327, C328, C329, C330: footprint (none) -> Capacitors_SMD:C_0805
- C305, C306, C307, C308, C309, C310, C311, C312, C313, C314, C315, C316, C317, C318, C319, C320, C321, C322, C323, C324, C325, C331, C332: footprint (none) -> Capacitors_SMD:C_0402
- D2, D3: footprint (none) -> Diodes_SMD:D_0805
- D4: footprint (none) -> Diodes_SMD:D_SOD-123
- D5, D6: footprint (none) -> Diodes_SMD:D_SOD-323
- FB10, FB11, FB12, FB13, FB3, FB4, FB5, FB6, FB7, FB8, FB9: footprint (none) -> Resistors_SMD:R_0603
- J5: footprint (none) -> SMD_Packages:Conn-20
- L2: footprint (none) -> Resistors_SMD:R_1210
- R301, R302, R303, R304, R305, R306, R307, R308, R309, R310: footprint (none) -> Resistors_SMD:R_0402
- U4: footprint (none) -> Housings_QFP:TQFP-100-1EP_14x14mm_Pitch0.5mm
- U5: footprint (none) -> TO_SOT_Packages_SMD:TSOT-23-5
- U7: footprint (none) -> Housings_SOIC:SOIC-20W_7.5x12.8mm_Pitch1.27mm
- Y2: footprint (none) -> Crystals:Resonator_SMD_muRata_CDSCB-2pin_4.5x2.0mm

Commit message: Revise component numbering and footprints
Parts:
- FB3, FB4, FB5, FB6, FB7, FB9: value Ferrite_Bead_Small -> BLM18RK601SN1D
- renumbered D2 to D301, D3 to D302, D4 to D303, D5 to D304, D6 to D305
Changed lines of the file:
@@
 P 8900 6100
 F 0 "FB9" V 8755 6100 50  0000 C CNN
-F 1 "Ferrite_Bead_Small" V 8754 6100 50  0001 C CNN
+F 1 "BLM18RK601SN1D" V 8754 6100 50  0001 C CNN
 F 2 "Resistors_SMD:R_0603" V 8830 6100 50  0001 C CNN
 F 3 "~" H 8900 6100 50  0001 C CNN
@@
 P 12550 1200
 F 0 "FB7" H 12650 1200 50  0000 L CNN
-F 1 "Ferrite_Bead_Small" H 12650 1155 50  0001 L CNN
+F 1 "BLM18RK601SN1D" H 12650 1155 50  0001 L CNN
 F 2 "Resistors_SMD:R_0603" V 12480 1200 50  0001 C CNN
 F 3 "~" H 12550 1200 50  0001 C CNN
@@
 	13350 1400 12550 1400
 $Comp
-L Device:LED D2
+L Device:LED D301
 U 1 1 5BC576DB
 P 13700 1700
-F 0 "D2" H 13692 1445 50  0000 C CNN
+F 0 "D301" H 13692 1445 50  0000 C CNN
 F 1 "RED" H 13692 1536 50  0000 C CNN
 F 2 "Diodes_SMD:D_0805" H 13700 1700 50  0001 C CNN
@@
 	8900 8950 9200 8950
 $Comp
-L Device:LED D3
+L Device:LED D302
 U 1 1 5BCEEB6C
 P 9500 8100
-F 0 "D3" V 9538 7983 50  0000 R CNN
+F 0 "D302" V 9538 7983 50  0000 R CNN
 F 1 "BLUE" V 9447 7983 50  0000 R CNN
 F 2 "Diodes_SMD:D_0805" H 9500 8100 50  0001 C CNN
@@
 $EndComp
 $Comp
-L Device:D D4
+L Device:D D303
 U 1 1 5BD9AD8A
 P 13400 6900
-F 0 "D4" H 13400 6684 50  0000 C CNN
+F 0 "D303" H 13400 6684 50  0000 C CNN
 F 1 "MBR0540" H 13400 6775 50  0000 C CNN
 F 2 "Diodes_SMD:D_SOD-123" H 13400 6900 50  0001 C CNN
@@
 	13200 7600 13200 6900
 $Comp
-L Device:D D5
+L Device:D D304
 U 1 1 5BDEB2E3
 P 14300 7100
-F 0 "D5" V 14254 7179 50  0000 L CNN
+F 0 "D304" V 14254 7179 50  0000 L CNN
 F 1 "MM3Z24VT1G" V 14345 7179 50  0000 L CNN
 F 2 "Diodes_SMD:D_SOD-323" H 14300 7100 50  0001 C CNN
@@
 	11650 7500 11750 7500
 $Comp
-L Device:D_Small D6
+L Device:D_Small D305
 U 1 1 5BE9FE0C
 P 12050 8100
-F 0 "D6" V 12096 8032 50  0000 R CNN
+F 0 "D305" V 12096 8032 50  0000 R CNN
 F 1 "1N4148" V 12005 8032 50  0000 R CNN
 F 2 "Diodes_SMD:D_SOD-323" V 12050 8100 50  0001 C CNN
@@
 P 3650 5600
 F 0 "FB6" V 3505 5600 50  0000 C CNN
-F 1 "Ferrite_Bead_Small" V 3504 5600 50  0001 C CNN
+F 1 "BLM18RK601SN1D" V 3504 5600 50  0001 C CNN
 F 2 "Resistors_SMD:R_0603" V 3580 5600 50  0001 C CNN
 F 3 "~" H 3650 5600 50  0001 C CNN
@@
 P 3650 5150
 F 0 "FB5" V 3505 5150 50  0000 C CNN
-F 1 "Ferrite_Bead_Small" V 3504 5150 50  0001 C CNN
+F 1 "BLM18RK601SN1D" V 3504 5150 50  0001 C CNN
 F 2 "Resistors_SMD:R_0603" V 3580 5150 50  0001 C CNN
 F 3 "~" H 3650 5150 50  0001 C CNN
@@
 P 3650 4600
 F 0 "FB4" V 3505 4600 50  0000 C CNN
-F 1 "Ferrite_Bead_Small" V 3504 4600 50  0001 C CNN
+F 1 "BLM18RK601SN1D" V 3504 4600 50  0001 C CNN
 F 2 "Resistors_SMD:R_0603" V 3580 4600 50  0001 C CNN
 F 3 "~" H 3650 4600 50  0001 C CNN
@@
 P 3650 4250
 F 0 "FB3" V 3505 4250 50  0000 C CNN
-F 1 "Ferrite_Bead_Small" V 3504 4250 50  0001 C CNN
+F 1 "BLM18RK601SN1D" V 3504 4250 50  0001 C CNN
 F 2 "Resistors_SMD:R_0603" V 3580 4250 50  0001 C CNN
 F 3 "~" H 3650 4250 50  0001 C CNN

Commit message: Add netlist to PCB design
Parts:
- J6: footprint (none) -> Connectors:HE10-40D
Changed lines of the file:
@@
 F 0 "J6" H 10480 3592 50  0000 L CNN
 F 1 "FFC-40" H 10480 3501 50  0000 L CNN
-F 2 "" H 10400 3600 50  0001 C CNN
+F 2 "Connectors:HE10-40D" H 10400 3600 50  0001 C CNN
 F 3 "~" H 10400 3600 50  0001 C CNN
 	1    10400 3600
