File: hardware/mainboard/chartreuse/chartreuse-power.sch (KiCad schematic (older format))
At the start: 16 parts, among them Q1 MMUN2133LT1G, U1 MCP73871, U2 TPS61090

Commit message: Add project-specific component library
Create components for TFP401, AR1100, 24LC02, USB2422, and FAN5333. In addition, add schematic sheets for HDMI and USB subsections.
Parts:
- added R? (x2): 100K, symbol Device:R
- added R?: 1K, symbol Device:R
- added R?: 15K, symbol Device:R
- added R?: 270K, symbol Device:R
- C101: renamed from C?; value C -> 10uF
Connections:
- wire segments 78 -> 93
Changed lines of the file:
@@
 EESchema Schematic File Version 4
+LIBS:chartreuse-cache
 EELAYER 26 0
 EELAYER END
 $Descr A 11000 8500
 encoding utf-8
-Sheet 2 2
+Sheet 2 4
 Title ""
 Date "2018-06-10"
@@
 Comment4 ""
 $EndDescr
-Text HLabel 4700 1450 0    50   Input ~ 0
+Text HLabel 3200 1450 0    50   Input ~ 0
 VCHARGE
 Text HLabel 8000 2300 2    50   Input ~ 0
@@
 Connection ~ 6800 2300
 $Comp
-L Device:C C?
+L Device:C C101
 U 1 1 5B21277E
 P 7900 2550
-F 0 "C?" H 8015 2596 50  0000 L CNN
-F 1 "C" H 8015 2505 50  0000 L CNN
+F 0 "C101" H 8015 2596 50  0000 L CNN
+F 1 "10uF" H 8015 2505 50  0000 L CNN
 F 2 "" H 7938 2400 50  0001 C CNN
 F 3 "~" H 7900 2550 50  0001 C CNN
@@
 $EndComp
 Wire Wire Line
-	4700 1450 5200 1450
+	3200 1450 4100 1450
 Wire Wire Line
 	6000 1450 6000 1700
@@
 	9150 4650 9150 4900
 $Comp
-L power:GND #PWR?
+L power:GND #PWR0127
 U 1 1 5B230E98
 P 9150 6200
-F 0 "#PWR?" H 9150 5950 50  0001 C CNN
+F 0 "#PWR0127" H 9150 5950 50  0001 C CNN
 F 1 "GND" H 9155 6027 50  0000 C CNN
 F 2 "" H 9150 6200 50  0001 C CNN
@@
 Wire Wire Line
 	5200 1450 6000 1450
+$Comp
+L Device:R R?
+U 1 1 5B5B7B16
+P 4650 3550
+F 0 "R?" H 4720 3596 50  0000 L CNN
+F 1 "100K" H 4720 3505 50  0000 L CNN
+F 2 "" V 4580 3550 50  0001 C CNN
+F 3 "~" H 4650 3550 50  0001 C CNN
+	1    4650 3550
+	1    0    0    -1
+$EndComp
+$Comp
+L Device:R R?
+U 1 1 5B5B7B72
+P 4400 3550
+F 0 "R?" H 4470 3596 50  0000 L CNN
+F 1 "1K" H 4470 3505 50  0000 L CNN
+F 2 "" V 4330 3550 50  0001 C CNN
+F 3 "~" H 4400 3550 50  0001 C CNN
+	1    4400 3550
+	1    0    0    -1
+$EndComp
+Wire Wire Line
+	4400 3400 4400 2400
+Wire Wire Line
+	4400 2400 5300 2400
+Wire Wire Line
+	4650 3400 4650 2600
+Wire Wire Line
+	4650 2600 5300 2600
+$Comp
+L power:GND #PWR?
+U 1 1 5B5BB2AF
+P 4650 3800
+F 0 "#PWR?" H 4650 3550 50  0001 C CNN
+F 1 "GND" H 4655 3627 50  0000 C CNN
+F 2 "" H 4650 3800 50  0001 C CNN
+F 3 "" H 4650 3800 50  0001 C CNN
+	1    4650 3800
+	1    0    0    -1
+$EndComp
+$Comp
+L power:GND #PWR?
+U 1 1 5B5BB41B
+P 4400 3800
+F 0 "#PWR?" H 4400 3550 50  0001 C CNN
+F 1 "GND" H 4405 3627 50  0000 C CNN
+F 2 "" H 4400 3800 50  0001 C CNN
+F 3 "" H 4400 3800 50  0001 C CNN
+	1    4400 3800
+	1    0    0    -1
+$EndComp
+Wire Wire Line
+	4400 3800 4400 3700
+$Comp
+L Device:R R?
+U 1 1 5B5BD0DC
+P 5000 3550
+F 0 "R?" H 5070 3596 50  0000 L CNN
+F 1 "15K" H 5070 3505 50  0000 L CNN
+F 2 "" V 4930 3550 50  0001 C CNN
+F 3 "~" H 5000 3550 50  0001 C CNN
+	1    5000 3550
+	1    0    0    -1
+$EndComp
+Wire Wire Line
+	4650 3700 4650 3800
+$Comp
+L power:GND #PWR?
+U 1 1 5B5C0BAF
+P 5000 3800
+F 0 "#PWR?" H 5000 3550 50  0001 C CNN
+F 1 "GND" H 5005 3627 50  0000 C CNN
+F 2 "" H 5000 3800 50  0001 C CNN
+F 3 "" H 5000 3800 50  0001 C CNN
+	1    5000 3800
+	1    0    0    -1
+$EndComp
+Wire Wire Line
+	5000 3800 5000 3700
+Wire Wire Line
+	5000 3400 5000 2800
+Wire Wire Line
+	5000 2800 5300 2800
+$Comp
+L Device:R R?
+U 1 1 5B5C49B1
+P 4100 3550
+F 0 "R?" H 4170 3596 50  0000 L CNN
+F 1 "100K" H 4170 3505 50  0000 L CNN
+F 2 "" V 4030 3550 50  0001 C CNN
+F 3 "~" H 4100 3550 50  0001 C CNN
+	1    4100 3550
+	1    0    0    -1
+$EndComp
+$Comp
+L Device:R R?
+U 1 1 5B5C6988
+P 4100 1700
+F 0 "R?" H 4170 1746 50  0000 L CNN
+F 1 "270K" H 4170 1655 50  0000 L CNN
+F 2 "" V 4030 1700 50  0001 C CNN
+F 3 "~" H 4100 1700 50  0001 C CNN
+	1    4100 1700
+	1    0    0    -1
+$EndComp
+Wire Wire Line
+	4100 1850 4100 2000
+Wire Wire Line
+	4100 1550 4100 1450
+Connection ~ 4100 1450
+Wire Wire Line
+	4100 1450 5200 1450
+Wire Wire Line
+	4100 2000 5300 2000
+Connection ~ 4100 2000
+Wire Wire Line
+	4100 2000 4100 3400
+$Comp
+L power:GND #PWR?
+U 1 1 5B5D310D
+P 4100 3800
+F 0 "#PWR?" H 4100 3550 50  0001 C CNN
+F 1 "GND" H 4105 3627 50  0000 C CNN
+F 2 "" H 4100 3800 50  0001 C CNN
+F 3 "" H 4100 3800 50  0001 C CNN
+	1    4100 3800
+	1    0    0    -1
+$EndComp
+Wire Wire Line
+	4100 3800 4100 3700
 $EndSCHEMATC

Commit message: Add component references
Parts:
- removed D1: LED_ALT, symbol Device:LED_ALT
- added D1: LED, symbol Device:LED
- gave numbers to parts that had none: 14
Changed lines of the file:
@@
 encoding utf-8
 Sheet 2 4
-Title ""
-Date "2018-06-10"
-Rev ""
+Title "Chartreuse Main Board"
+Date "2018-09-21"
+Rev "0.9"
 Comp ""
 Comment1 ""
@@
 	3850 6950 3850 7050
 $Comp
-L Device:R R?
+L Device:R R108
 U 1 1 5B1E04C1
 P 4700 6000
-F 0 "R?" H 4770 6046 50  0000 L CNN
+F 0 "R108" H 4770 6046 50  0000 L CNN
 F 1 "1.87M" H 4770 5955 50  0000 L CNN
 F 2 "" V 4630 6000 50  0001 C CNN
@@
 	6050 5650 5600 5650
 $Comp
-L Device:C C?
+L Device:C C104
 U 1 1 5B1E067A
 P 5150 6000
-F 0 "C?" H 5265 6046 50  0000 L CNN
+F 0 "C104" H 5265 6046 50  0000 L CNN
 F 1 "2.2uF" H 5265 5955 50  0000 L CNN
 F 2 "" H 5188 5850 50  0001 C CNN
@@
 Connection ~ 4150 5950
 $Comp
-L Device:R R?
+L Device:R R109
 U 1 1 5B1E0B83
 P 4700 6500
-F 0 "R?" H 4770 6546 50  0000 L CNN
+F 0 "R109" H 4770 6546 50  0000 L CNN
 F 1 "200K" H 4770 6455 50  0000 L CNN
 F 2 "" V 4630 6500 50  0001 C CNN
@@
 	4500 6350 4050 6350
 $Comp
-L Device:CP1 C?
+L Device:CP1 C105
 U 1 1 5B1E2B0B
 P 5600 6000
-F 0 "C?" H 5715 6046 50  0000 L CNN
+F 0 "C105" H 5715 6046 50  0000 L CNN
 F 1 "100uF" H 5715 5955 50  0000 L CNN
 F 2 "" H 5600 6000 50  0001 C CNN
@@
 	8350 5100 8800 5100
 $Comp
-L Device:R R?
+L Device:R R106
 U 1 1 5B1E51C1
 P 2250 6100
-F 0 "R?" H 2320 6146 50  0000 L CNN
+F 0 "R106" H 2320 6146 50  0000 L CNN
 F 1 "1.87M" H 2320 6055 50  0000 L CNN
 F 2 "" V 2180 6100 50  0001 C CNN
@@
 $EndComp
 $Comp
-L Device:R R?
+L Device:R R107
 U 1 1 5B1E51C7
 P 2250 6600
-F 0 "R?" H 2320 6646 50  0000 L CNN
+F 0 "R107" H 2320 6646 50  0000 L CNN
 F 1 "340K" H 2320 6555 50  0000 L CNN
 F 2 "" V 2180 6600 50  0001 C CNN
@@
 	2250 6850 2250 6750
 $Comp
-L Device:C C?
+L Device:C C103
 U 1 1 5B1E8F52
 P 1850 6100
-F 0 "C?" H 1965 6146 50  0000 L CNN
+F 0 "C103" H 1965 6146 50  0000 L CNN
 F 1 "0.1uF" H 1965 6055 50  0000 L CNN
 F 2 "" H 1888 5950 50  0001 C CNN
@@
 $EndComp
 $Comp
-L Device:C C?
+L Device:C C102
 U 1 1 5B1E8FCA
 P 1400 6100
-F 0 "C?" H 1515 6146 50  0000 L CNN
+F 0 "C102" H 1515 6146 50  0000 L CNN
 F 1 "10uF" H 1515 6055 50  0000 L CNN
 F 2 "" H 1438 5950 50  0001 C CNN
@@
 	7200 2000 6700 2000
 $Comp
-L Device:R R?
+L Device:R R110
 U 1 1 5B223150
 P 9150 5550
-F 0 "R?" H 9220 5596 50  0000 L CNN
+F 0 "R110" H 9220 5596 50  0000 L CNN
 F 1 "1K" H 9220 5505 50  0000 L CNN
 F 2 "" V 9080 5550 50  0001 C CNN
@@
 	1    0    0    -1
 $EndComp
-$Comp
-L Device:LED_ALT D1
-U 1 1 5B23233F
-P 9150 5950
-F 0 "D1" V 9188 5832 50  0000 R CNN
-F 1 "LED_ALT" V 9097 5832 50  0000 R CNN
-F 2 "" H 9150 5950 50  0001 C CNN
-F 3 "~" H 9150 5950 50  0001 C CNN
-	1    9150 5950
-	0    -1   -1   0
-$EndComp
 Wire Wire Line
 	9150 5800 9150 5700
@@
 	5200 1450 6000 1450
 $Comp
-L Device:R R?
+L Device:R R104
 U 1 1 5B5B7B16
 P 4650 3550
-F 0 "R?" H 4720 3596 50  0000 L CNN
+F 0 "R104" H 4720 3596 50  0000 L CNN
 F 1 "100K" H 4720 3505 50  0000 L CNN
 F 2 "" V 4580 3550 50  0001 C CNN
@@
 $EndComp
 $Comp
-L Device:R R?
+L Device:R R103
 U 1 1 5B5B7B72
 P 4400 3550
-F 0 "R?" H 4470 3596 50  0000 L CNN
+F 0 "R103" H 4470 3596 50  0000 L CNN
 F 1 "1K" H 4470 3505 50  0000 L CNN
 F 2 "" V 4330 3550 50  0001 C CNN
@@
 	4400 3800 4400 3700
 $Comp
-L Device:R R?
+L Device:R R105
 U 1 1 5B5BD0DC
 P 5000 3550
-F 0 "R?" H 5070 3596 50  0000 L CNN
+F 0 "R105" H 5070 3596 50  0000 L CNN
 F 1 "15K" H 5070 3505 50  0000 L CNN
 F 2 "" V 4930 3550 50  0001 C CNN
@@
 	5000 2800 5300 2800
 $Comp
-L Device:R R?
+L Device:R R102
 U 1 1 5B5C49B1
 P 4100 3550
-F 0 "R?" H 4170 3596 50  0000 L CNN
+F 0 "R102" H 4170 3596 50  0000 L CNN
 F 1 "100K" H 4170 3505 50  0000 L CNN
 F 2 "" V 4030 3550 50  0001 C CNN
@@
 $EndComp
 $Comp
-L Device:R R?
+L Device:R R101
 U 1 1 5B5C6988
 P 4100 1700
-F 0 "R?" H 4170 1746 50  0000 L CNN
+F 0 "R101" H 4170 1746 50  0000 L CNN
 F 1 "270K" H 4170 1655 50  0000 L CNN
 F 2 "" V 4030 1700 50  0001 C CNN
@@
 Wire Wire Line
 	4100 3800 4100 3700
+$Comp
+L Device:LED D1
+U 1 1 5BA81F14
+P 9150 5950
+F 0 "D1" V 9188 5833 50  0000 R CNN
+F 1 "LED" V 9097 5833 50  0000 R CNN
+F 2 "" H 9150 5950 50  0001 C CNN
+F 3 "~" H 9150 5950 50  0001 C CNN
+	1    9150 5950
+	0    -1   -1   0
+$EndComp
 $EndSCHEMATC

Commit message: Schematic DRC check
Parts:
- gave numbers to parts that had none: 1
- renumbered R108 to R109, R109 to R110, R110 to R111
Connections:
- no-connect marks 1 -> 3

Commit message: Preliminary assign footprints
Parts:
- C101: footprint (none) -> Capacitors_SMD:CP_Elec_4x5.8
- C102, C104: footprint (none) -> Capacitors_SMD:C_0805
- C103: footprint (none) -> Capacitors_SMD:C_0402
- C105: footprint (none) -> Capacitors_SMD:CP_Elec_5x5.8
- D1: footprint (none) -> Diodes_SMD:D_0805
- L1: footprint (none) -> Inductors_SMD:L_Taiyo-Yuden_NR-40xx_HandSoldering
- Q1: footprint (none) -> TO_SOT_Packages_SMD:SOT-23
- R101, R102, R103, R104, R105, R106, R107, R108, R109, R110, R111: footprint (none) -> Resistors_SMD:R_0402
Changed lines of the file:
@@
 F 0 "R109" H 4770 6046 50  0000 L CNN
 F 1 "1.87M" H 4770 5955 50  0000 L CNN
-F 2 "" V 4630 6000 50  0001 C CNN
+F 2 "Resistors_SMD:R_0402" V 4630 6000 50  0001 C CNN
 F 3 "~" H 4700 6000 50  0001 C CNN
 	1    4700 6000
@@
 F 0 "C104" H 5265 6046 50  0000 L CNN
 F 1 "2.2uF" H 5265 5955 50  0000 L CNN
-F 2 "" H 5188 5850 50  0001 C CNN
+F 2 "Capacitors_SMD:C_0805" H 5188 5850 50  0001 C CNN
 F 3 "~" H 5150 6000 50  0001 C CNN
 	1    5150 6000
@@
 F 0 "R110" H 4770 6546 50  0000 L CNN
 F 1 "200K" H 4770 6455 50  0000 L CNN
-F 2 "" V 4630 6500 50  0001 C CNN
+F 2 "Resistors_SMD:R_0402" V 4630 6500 50  0001 C CNN
 F 3 "~" H 4700 6500 50  0001 C CNN
 	1    4700 6500
@@
 F 0 "C105" H 5715 6046 50  0000 L CNN
 F 1 "100uF" H 5715 5955 50  0000 L CNN
-F 2 "" H 5600 6000 50  0001 C CNN
+F 2 "Capacitors_SMD:CP_Elec_5x5.8" H 5600 6000 50  0001 C CNN
 F 3 "~" H 5600 6000 50  0001 C CNN
 	1    5600 6000
@@
 F 0 "Q1" H 9237 5054 50  0000 L CNN
 F 1 "MMUN2133LT1G" H 9237 5145 50  0000 L CNN
-F 2 "" H 9050 5100 50  0001 L CNN
+F 2 "TO_SOT_Packages_SMD:SOT-23" H 9050 5100 50  0001 L CNN
 F 3 "" H 9050 5100 50  0001 L CNN
 	1    9050 5100
@@
 F 0 "R106" H 2320 6146 50  0000 L CNN
 F 1 "1.87M" H 2320 6055 50  0000 L CNN
-F 2 "" V 2180 6100 50  0001 C CNN
+F 2 "Resistors_SMD:R_0402" V 2180 6100 50  0001 C CNN
 F 3 "~" H 2250 6100 50  0001 C CNN
 	1    2250 6100
@@
 F 0 "R107" H 2320 6646 50  0000 L CNN
 F 1 "340K" H 2320 6555 50  0000 L CNN
-F 2 "" V 2180 6600 50  0001 C CNN
+F 2 "Resistors_SMD:R_0402" V 2180 6600 50  0001 C CNN
 F 3 "~" H 2250 6600 50  0001 C CNN
 	1    2250 6600
@@
 F 0 "L1" V 2840 5650 50  0000 C CNN
 F 1 "6.8uH" V 2749 5650 50  0000 C CNN
-F 2 "" H 2650 5650 50  0001 C CNN
+F 2 "Inductors_SMD:L_Taiyo-Yuden_NR-40xx_HandSoldering" H 2650 5650 50  0001 C CNN
 F 3 "~" H 2650 5650 50  0001 C CNN
 	1    2650 5650
@@
 F 0 "C103" H 1965 6146 50  0000 L CNN
 F 1 "0.1uF" H 1965 6055 50  0000 L CNN
-F 2 "" H 1888 5950 50  0001 C CNN
+F 2 "Capacitors_SMD:C_0402" H 1888 5950 50  0001 C CNN
 F 3 "~" H 1850 6100 50  0001 C CNN
 	1    1850 6100
@@
 F 0 "C102" H 1515 6146 50  0000 L CNN
 F 1 "10uF" H 1515 6055 50  0000 L CNN
-F 2 "" H 1438 5950 50  0001 C CNN
+F 2 "Capacitors_SMD:C_0805" H 1438 5950 50  0001 C CNN
 F 3 "~" H 1400 6100 50  0001 C CNN
 	1    1400 6100
@@
 F 0 "R108" H 3120 4796 50  0000 L CNN
 F 1 "200K" H 3120 4705 50  0000 L CNN
-F 2 "" V 2980 4750 50  0001 C CNN
+F 2 "Resistors_SMD:R_0402" V 2980 4750 50  0001 C CNN
 F 3 "~" H 3050 4750 50  0001 C CNN
 	1    3050 4750
@@
 F 0 "C101" H 8365 2596 50  0000 L CNN
 F 1 "10uF" H 8365 2505 50  0000 L CNN
-F 2 "" H 8288 2400 50  0001 C CNN
+F 2 "Capacitors_SMD:CP_Elec_4x5.8" H 8288 2400 50  0001 C CNN
 F 3 "~" H 8250 2550 50  0001 C CNN
 	1    8250 2550
@@
 F 0 "R111" H 9220 5596 50  0000 L CNN
 F 1 "1K" H 9220 5505 50  0000 L CNN
-F 2 "" V 9080 5550 50  0001 C CNN
+F 2 "Resistors_SMD:R_0402" V 9080 5550 50  0001 C CNN
 F 3 "~" H 9150 5550 50  0001 C CNN
 	1    9150 5550
@@
 F 0 "R104" H 4920 3596 50  0000 L CNN
 F 1 "100K" H 4920 3505 50  0000 L CNN
-F 2 "" V 4780 3550 50  0001 C CNN
+F 2 "Resistors_SMD:R_0402" V 4780 3550 50  0001 C CNN
 F 3 "~" H 4850 3550 50  0001 C CNN
 	1    4850 3550
@@
 F 0 "R103" H 4570 3596 50  0000 L CNN
 F 1 "1K" H 4570 3505 50  0000 L CNN
-F 2 "" V 4430 3550 50  0001 C CNN
+F 2 "Resistors_SMD:R_0402" V 4430 3550 50  0001 C CNN
 F 3 "~" H 4500 3550 50  0001 C CNN
 	1    4500 3550
@@
 F 0 "R105" H 5270 3596 50  0000 L CNN
 F 1 "15K" H 5270 3505 50  0000 L CNN
-F 2 "" V 5130 3550 50  0001 C CNN
+F 2 "Resistors_SMD:R_0402" V 5130 3550 50  0001 C CNN
 F 3 "~" H 5200 3550 50  0001 C CNN
 	1    5200 3550
@@
 F 0 "R102" H 4220 3596 50  0000 L CNN
 F 1 "100K" H 4220 3505 50  0000 L CNN
-F 2 "" V 4080 3550 50  0001 C CNN
+F 2 "Resistors_SMD:R_0402" V 4080 3550 50  0001 C CNN
 F 3 "~" H 4150 3550 50  0001 C CNN
 	1    4150 3550
@@
 F 0 "R101" H 4220 1746 50  0000 L CNN
 F 1 "270K" H 4220 1655 50  0000 L CNN
-F 2 "" V 4080 1700 50  0001 C CNN
+F 2 "Resistors_SMD:R_0402" V 4080 1700 50  0001 C CNN
 F 3 "~" H 4150 1700 50  0001 C CNN
 	1    4150 1700
@@
 F 0 "D1" V 9188 5833 50  0000 R CNN
 F 1 "LED" V 9097 5833 50  0000 R CNN
-F 2 "" H 9150 5950 50  0001 C CNN
+F 2 "Diodes_SMD:D_0805" H 9150 5950 50  0001 C CNN
 F 3 "~" H 9150 5950 50  0001 C CNN
 	1    9150 5950

Commit message: Revise component numbering and footprints
Parts:
- added D101: ORANGE, Diodes_SMD:D_0805, symbol Device:LED
- added D102: GREEN, Diodes_SMD:D_0805, symbol Device:LED
- added R112, R113: 1K, Resistors_SMD:R_0402, symbol Device:R
- added SW1: SW_SPDT, symbol Switch:SW_SPDT
- D103: renamed from D1; value LED -> RED
Connections:
- wire segments 93 -> 106
- no-connect marks 3 -> 2
Changed lines of the file:
@@
 Text HLabel 3250 1450 0    50   Input ~ 0
 VCHARGE
-Text HLabel 8350 2300 2    50   Input ~ 0
+Text HLabel 7600 2300 2    50   Input ~ 0
 VLIPO
 Text HLabel 6050 5650 2    50   Output ~ 0
@@
 L Transistor_BJT:DTA143Z Q1
 U 1 1 5B1E317F
-P 9050 5100
-F 0 "Q1" H 9237 5054 50  0000 L CNN
-F 1 "MMUN2133LT1G" H 9237 5145 50  0000 L CNN
-F 2 "TO_SOT_Packages_SMD:SOT-23" H 9050 5100 50  0001 L CNN
-F 3 "" H 9050 5100 50  0001 L CNN
-	1    9050 5100
+P 9500 4300
+F 0 "Q1" H 9687 4254 50  0000 L CNN
+F 1 "MMUN2133LT1G" H 9687 4345 50  0000 L CNN
+F 2 "TO_SOT_Packages_SMD:SOT-23" H 9500 4300 50  0001 L CNN
+F 3 "" H 9500 4300 50  0001 L CNN
+	1    9500 4300
 	1    0    0    1
 $EndComp
@@
 Connection ~ 4150 5850
 Connection ~ 4700 5650
-Text Label 8350 5100 0    50   ~ 0
+Text Label 8800 4300 0    50   ~ 0
 LOW_BATT
 Wire Wire Line
-	8350 5100 8800 5100
+	8800 4300 9250 4300
 $Comp
 L Device:R R106
@@
 	7150 2300 7050 2300
 Wire Wire Line
-	7150 2300 8250 2300
+	7150 2300 7500 2300
 Connection ~ 7150 2300
 $Comp
 L Device:C C101
 U 1 1 5B21277E
-P 8250 2550
-F 0 "C101" H 8365 2596 50  0000 L CNN
-F 1 "10uF" H 8365 2505 50  0000 L CNN
-F 2 "Capacitors_SMD:CP_Elec_4x5.8" H 8288 2400 50  0001 C CNN
-F 3 "~" H 8250 2550 50  0001 C CNN
-	1    8250 2550
-	1    0    0    -1
-$EndComp
-Wire Wire Line
-	8250 2400 8250 2300
-Connection ~ 8250 2300
-Wire Wire Line
-	8250 2300 8350 2300
-Wire Wire Line
-	8250 2700 8250 2800
+P 7500 2550
+F 0 "C101" H 7615 2596 50  0000 L CNN
+F 1 "10uF" H 7615 2505 50  0000 L CNN
+F 2 "Capacitors_SMD:CP_Elec_4x5.8" H 7538 2400 50  0001 C CNN
+F 3 "~" H 7500 2550 50  0001 C CNN
+	1    7500 2550
+	1    0    0    -1
+$EndComp
+Wire Wire Line
+	7500 2400 7500 2300
+Connection ~ 7500 2300
+Wire Wire Line
+	7500 2300 7600 2300
+Wire Wire Line
+	7500 2700 7500 3200
 $Comp
 L power:GND #PWR0121
 U 1 1 5B216839
-P 8250 2800
-F 0 "#PWR0121" H 8250 2550 50  0001 C CNN
-F 1 "GND" H 8255 2627 50  0000 C CNN
-F 2 "" H 8250 2800 50  0001 C CNN
-F 3 "" H 8250 2800 50  0001 C CNN
-	1    8250 2800
+P 7500 3200
+F 0 "#PWR0121" H 7500 2950 50  0001 C CNN
+F 1 "GND" H 7505 3027 50  0000 C CNN
+F 2 "" H 7500 3200 50  0001 C CNN
+F 3 "" H 7500 3200 50  0001 C CNN
+	1    7500 3200
 	1    0    0    -1
 $EndComp
@@
 	6350 3600 6350 3500
 NoConn ~ 7050 2800
-Text Label 7550 2000 2    50   ~ 0
+Text Label 7500 2000 2    50   ~ 0
 VBAT
 Wire Wire Line
-	7550 2000 7050 2000
+	7500 2000 7050 2000
 $Comp
 L Device:R R111
 U 1 1 5B223150
-P 9150 5550
-F 0 "R111" H 9220 5596 50  0000 L CNN
-F 1 "1K" H 9220 5505 50  0000 L CNN
-F 2 "Resistors_SMD:R_0402" V 9080 5550 50  0001 C CNN
-F 3 "~" H 9150 5550 50  0001 C CNN
-	1    9150 5550
-	1    0    0    -1
-$EndComp
-Text Label 9150 4650 3    50   ~ 0
+P 9600 4750
+F 0 "R111" H 9670 4796 50  0000 L CNN
+F 1 "1K" H 9670 4705 50  0000 L CNN
+F 2 "Resistors_SMD:R_0402" V 9530 4750 50  0001 C CNN
+F 3 "~" H 9600 4750 50  0001 C CNN
+	1    9600 4750
+	1    0    0    -1
+$EndComp
+Text Label 9600 3850 3    50   ~ 0
 VBAT
 Wire Wire Line
-	9150 5400 9150 5300
-Wire Wire Line
-	9150 4650 9150 4900
+	9600 4600 9600 4500
+Wire Wire Line
+	9600 3850 9600 4100
 $Comp
 L power:GND #PWR0127
 U 1 1 5B230E98
-P 9150 6200
-F 0 "#PWR0127" H 9150 5950 50  0001 C CNN
-F 1 "GND" H 9155 6027 50  0000 C CNN
-F 2 "" H 9150 6200 50  0001 C CNN
-F 3 "" H 9150 6200 50  0001 C CNN
-	1    9150 6200
-	1    0    0    -1
-$EndComp
-Wire Wire Line
-	9150 5800 9150 5700
-Wire Wire Line
-	9150 6100 9150 6200
+P 9600 5400
+F 0 "#PWR0127" H 9600 5150 50  0001 C CNN
+F 1 "GND" H 9605 5227 50  0000 C CNN
+F 2 "" H 9600 5400 50  0001 C CNN
+F 3 "" H 9600 5400 50  0001 C CNN
+	1    9600 5400
+	1    0    0    -1
+$EndComp
+Wire Wire Line
+	9600 5000 9600 4900
+Wire Wire Line
+	9600 5300 9600 5400
 Wire Wire Line
 	5650 2200 5550 2200
@@
 	4150 3800 4150 3700
 $Comp
-L Device:LED D1
+L Device:LED D103
 U 1 1 5BA81F14
-P 9150 5950
-F 0 "D1" V 9188 5833 50  0000 R CNN
-F 1 "LED" V 9097 5833 50  0000 R CNN
-F 2 "Diodes_SMD:D_0805" H 9150 5950 50  0001 C CNN
-F 3 "~" H 9150 5950 50  0001 C CNN
-	1    9150 5950
+P 9600 5150
+F 0 "D103" V 9638 5033 50  0000 R CNN
+F 1 "RED" V 9547 5033 50  0000 R CNN
+F 2 "Diodes_SMD:D_0805" H 9600 5150 50  0001 C CNN
+F 3 "~" H 9600 5150 50  0001 C CNN
+	1    9600 5150
 	0    -1   -1   0
 $EndComp
-NoConn ~ 7050 3000
-NoConn ~ 7050 3100
+Text Label 7900 5100 0    50   ~ 0
+PWR_EN
+$Comp
+L Switch:SW_SPDT SW1
+U 1 1 5BF90131
+P 8450 5100
+F 0 "SW1" H 8450 5385 50  0000 C CNN
+F 1 "SW_SPDT" H 8450 5294 50  0000 C CNN
+F 2 "" H 8450 5100 50  0001 C CNN
+F 3 "" H 8450 5100 50  0001 C CNN
+	1    8450 5100
+	1    0    0    -1
+$EndComp
+Wire Wire Line
+	7900 5100 8250 5100
+Wire Wire Line
+	8750 5300 8750 5200
+Wire Wire Line
+	8750 5200 8650 5200
+$Comp
+L power:GND #PWR0158
+U 1 1 5BF94E1F
+P 8750 5300
+F 0 "#PWR0158" H 8750 5050 50  0001 C CNN
+F 1 "GND" H 8755 5127 50  0000 C CNN
+F 2 "" H 8750 5300 50  0001 C CNN
+F 3 "" H 8750 5300 50  0001 C CNN
+	1    8750 5300
+	1    0    0    -1
+$EndComp
+NoConn ~ 8650 5000
+$Comp
+L Device:LED D101
+U 1 1 5BFCAC44
+P 8100 2000
+F 0 "D101" V 8138 1883 50  0000 R CNN
+F 1 "ORANGE" V 8047 1883 50  0000 R CNN
+F 2 "Diodes_SMD:D_0805" H 8100 2000 50  0001 C CNN
+F 3 "~" H 8100 2000 50  0001 C CNN
+	1    8100 2000
+	0    -1   -1   0
+$EndComp
+$Comp
+L Device:LED D102
+U 1 1 5BFCACAA
+P 8650 2000
+F 0 "D102" V 8688 1883 50  0000 R CNN
+F 1 "GREEN" V 8597 1883 50  0000 R CNN
+F 2 "Diodes_SMD:D_0805" H 8650 2000 50  0001 C CNN
+F 3 "~" H 8650 2000 50  0001 C CNN
+	1    8650 2000
+	0    -1   -1   0
+$EndComp
+$Comp
+L Device:R R112
+U 1 1 5BFCADA8
+P 8100 2400
+F 0 "R112" H 8170 2446 50  0000 L CNN
+F 1 "1K" H 8170 2355 50  0000 L CNN
+F 2 "Resistors_SMD:R_0402" V 8030 2400 50  0001 C CNN
+F 3 "~" H 8100 2400 50  0001 C CNN
+	1    8100 2400
+	1    0    0    -1
+$EndComp
+$Comp
+L Device:R R113
+U 1 1 5BFCAE10
+P 8650 2400
+F 0 "R113" H 8720 2446 50  0000 L CNN
+F 1 "1K" H 8720 2355 50  0000 L CNN
+F 2 "Resistors_SMD:R_0402" V 8580 2400 50  0001 C CNN
+F 3 "~" H 8650 2400 50  0001 C CNN
+	1    8650 2400
+	1    0    0    -1
+$EndComp
+Wire Wire Line
+	8100 2150 8100 2250
+Wire Wire Line
+	8650 2250 8650 2150
+Wire Wire Line
+	8100 1850 8100 1450
+Wire Wire Line
+	8100 1450 6350 1450
+Connection ~ 6350 1450
+Wire Wire Line
+	8650 1850 8650 1450
+Wire Wire Line
+	8650 1450 8100 1450
+Connection ~ 8100 1450
+Wire Wire Line
+	7050 3000 8100 3000
+Wire Wire Line
+	8100 3000 8100 2550
+Wire Wire Line
+	7050 3100 8650 3100
+Wire Wire Line
+	8650 3100 8650 2550
 $EndSCHEMATC

Commit message: Add netlist to PCB design
Parts:
- SW1: footprint (none) -> Buttons_Switches_THT:SW_CuK_OS102011MA1QN1_SPDT_Angled
- U1: footprint Package_DFN_QFN:QFN-20-1EP_4x4mm_P0.5mm_EP2.5x2.5mm -> Housings_DFN_QFN:QFN-20-1EP_4x4mm_Pitch0.5mm
- U2: footprint Package_DFN_QFN:QFN-16-1EP_4x4mm_P0.65mm_EP2.5x2.5mm -> Housings_DFN_QFN:QFN-16-1EP_4x4mm_Pitch0.65mm
Changed lines of the file:
@@
 F 0 "U1" H 5750 3450 50  0000 C CNN
 F 1 "MCP73871" H 5750 1750 50  0000 C CNN
-F 2 "Package_DFN_QFN:QFN-20-1EP_4x4mm_P0.5mm_EP2.5x2.5mm" H 6550 1700 50  0001 L CIN
+F 2 "Housings_DFN_QFN:QFN-20-1EP_4x4mm_Pitch0.5mm" H 6550 1700 50  0001 L CIN
 F 3 "http://www.mouser.com/ds/2/268/22090a-52174.pdf" H 6200 3150 50  0001 C CNN
 	1    6350 2600
@@
 F 0 "U2" H 3650 7075 50  0000 C CNN
 F 1 "TPS61090" H 3650 6984 50  0000 C CNN
-F 2 "Package_DFN_QFN:QFN-16-1EP_4x4mm_P0.65mm_EP2.5x2.5mm" H 2700 5300 50  0001 L CNN
+F 2 "Housings_DFN_QFN:QFN-16-1EP_4x4mm_Pitch0.65mm" H 2700 5300 50  0001 L CNN
 F 3 "http://www.ti.com/lit/ds/symlink/tps61090.pdf" H 3800 5200 50  0001 L CNN
 	1    3650 6350
@@
 F 0 "SW1" H 8450 5385 50  0000 C CNN
 F 1 "SW_SPDT" H 8450 5294 50  0000 C CNN
-F 2 "" H 8450 5100 50  0001 C CNN
+F 2 "Buttons_Switches_THT:SW_CuK_OS102011MA1QN1_SPDT_Angled" H 8450 5100 50  0001 C CNN
 F 3 "" H 8450 5100 50  0001 C CNN
 	1    8450 5100
