File: hardware/mainboard/chartreuse/chartreuse.kicad_pcb (KiCad board)
At the start: 2 copper layers, 100 x 79.8 mm, 0 parts

Commit message: Add netlist to PCB design
Parts:
- added C101: 10uF, Capacitors_SMD:CP_Elec_4x5.8, F.Cu at (102.9, 62.5)
- added C102: 10uF, Capacitors_SMD:C_0805, F.Cu at (92.4, 53.6)
- added C103: 0.1uF, Capacitors_SMD:C_0402, F.Cu at (102.1, 67.8)
- added C104: 2.2uF, Capacitors_SMD:C_0805, F.Cu at (65.8, 58.7)
- added C105: 100uF, Capacitors_SMD:CP_Elec_5x5.8, F.Cu at (113.5, 91.4)
- added C201: 0.1uF, Capacitors_SMD:C_0402, F.Cu at (124.1, 168.4)
- added C202: 0.1uF, Capacitors_SMD:C_0402, F.Cu at (140.3, 162.6)
- added C203: 0.1uF, Capacitors_SMD:C_0402, F.Cu at (145.6, 159.5)
- added C204: 10uF, Capacitors_SMD:C_0805, F.Cu at (131.3, 159.9)
- added C205: 1uF, Capacitors_SMD:C_0402, F.Cu at (140.1, 167.2)
- added C206: 6pF, Capacitors_SMD:C_0402, F.Cu at (149.9, 154.6)
- added C207: 6pF, Capacitors_SMD:C_0402, F.Cu at (144.8, 164.1)
- added C301: 10uF, Capacitors_SMD:C_0805, F.Cu at (241.6, 78.2)
- added C302: 10uF, Capacitors_SMD:C_0805, F.Cu at (220.5, 99.6)
- added C303: 10uF, Capacitors_SMD:C_0805, F.Cu at (225.0, 97.0)
- added C304: 10uF, Capacitors_SMD:C_0805, F.Cu at (241.6, 83.5)
- added C305: 0.1uF, Capacitors_SMD:C_0402, F.Cu at (250.5, 77.1)
- added C306: 0.1uF, Capacitors_SMD:C_0402, F.Cu at (246.1, 82.7)
- added C307: 0.1uF, Capacitors_SMD:C_0402, F.Cu at (237.0, 89.2)
- added C308: 0.1uF, Capacitors_SMD:C_0402, F.Cu at (225.1, 102.1)
- added C309: 0.1uF, Capacitors_SMD:C_0402, F.Cu at (241.7, 88.5)
- added C310: 0.1uF, Capacitors_SMD:C_0402, F.Cu at (259.6, 66.4)
- added C311: 0.1uF, Capacitors_SMD:C_0402, F.Cu at (255.2, 77.1)
- added C312: 0.1uF, Capacitors_SMD:C_0402, F.Cu at (246.4, 87.3)
- added C313: 0.1uF, Capacitors_SMD:C_0402, F.Cu at (234.5, 98.4)
- added C314: 0.1uF, Capacitors_SMD:C_0402, F.Cu at (229.8, 106.2)
- added C315: 0.1uF, Capacitors_SMD:C_0402, F.Cu at (234.0, 93.8)
- added C316: 0.1uF, Capacitors_SMD:C_0402, F.Cu at (225.1, 106.7)
- added C317: 0.1uF, Capacitors_SMD:C_0402, F.Cu at (229.8, 101.6)
- added C318: 103, Capacitors_SMD:C_0402, F.Cu at (264.1, 66.4)
- added C319: 103, Capacitors_SMD:C_0402, F.Cu at (264.1, 71.0)
- added C320: 103, Capacitors_SMD:C_0402, F.Cu at (234.3, 103.0)
- added C321: 103, Capacitors_SMD:C_0402, F.Cu at (250.9, 86.3)
- added C322: 0.1uF, Capacitors_SMD:C_0402, F.Cu at (241.7, 93.1)
- added C323: 0.1uF, Capacitors_SMD:C_0402, F.Cu at (250.8, 81.7)
- added C324: 12pF, Capacitors_SMD:C_0402, F.Cu at (246.2, 91.9)
- added C325: 12pF, Capacitors_SMD:C_0402, F.Cu at (259.8, 75.6)
- added C326: 10uF, Capacitors_SMD:C_0805, F.Cu at (245.6, 72.8)
- added C327: 10uF, Capacitors_SMD:C_0805, F.Cu at (213.4, 108.3)
- added C328: 10uF, Capacitors_SMD:C_0805, F.Cu at (229.4, 91.7)
- added C329: 1uF, Capacitors_SMD:C_0805, F.Cu at (255.0, 66.7)
- added C330: 1uF, Capacitors_SMD:C_0805, F.Cu at (236.8, 84.2)
- added C331: 0.1uF, Capacitors_SMD:C_0402, F.Cu at (259.6, 71.0)
- added C332: 0.1uF, Capacitors_SMD:C_0402, F.Cu at (239.2, 97.7)
- added C401: 10uF, Capacitors_SMD:CP_Elec_4x5.8, F.Cu at (243.2, 132.6)
- added C402: 10uF, Capacitors_SMD:CP_Elec_4x5.8, F.Cu at (250.3, 136.6)
- added D101: ORANGE, Diodes_SMD:D_0805, F.Cu at (80.5, 55.4)
- added D102: GREEN, Diodes_SMD:D_0805, F.Cu at (80.5, 52.3)
- added D103: RED, Diodes_SMD:D_0805, F.Cu at (80.5, 49.8)
- added D301: RED, Diodes_SMD:D_0805, F.Cu at (241.2, 72.9)
- added D302: BLUE, Diodes_SMD:D_0805, F.Cu at (225.0, 91.8)
- added D303: MBR0540, Diodes_SMD:D_SOD-123, F.Cu at (242.7, 67.2)
- added D304: MM3Z24VT1G, Diodes_SMD:D_SOD-323, F.Cu at (234.2, 78.7)
- added D305: 1N4148, Diodes_SMD:D_SOD-323, F.Cu at (249.6, 67.0)
- added FB1: BLM18RK601SN1D, Resistors_SMD:R_0603, F.Cu at (276.7, 66.6)
- added FB10: Ferrite_Bead_Small, Resistors_SMD:R_0603, F.Cu at (220.4, 66.6)
- added FB11: Ferrite_Bead_Small, Resistors_SMD:R_0603, F.Cu at (190.2, 100.4)
- added FB12: Ferrite_Bead_Small, Resistors_SMD:R_0603, F.Cu at (207.6, 87.6)
- added FB13: Ferrite_Bead_Small, Resistors_SMD:R_0603, F.Cu at (190.2, 95.4)
- added FB2: BLM18RK601SN1D, Resistors_SMD:R_0603, F.Cu at (128.9, 154.8)
- added FB3: BLM18RK601SN1D, Resistors_SMD:R_0603, F.Cu at (204.1, 105.4)
- added FB4: BLM18RK601SN1D, Resistors_SMD:R_0603, F.Cu at (204.7, 95.4)
- added FB5: BLM18RK601SN1D, Resistors_SMD:R_0603, F.Cu at (222.1, 86.6)
- added FB6: BLM18RK601SN1D, Resistors_SMD:R_0603, F.Cu at (222.1, 81.6)
- added FB7: BLM18RK601SN1D, Resistors_SMD:R_0603, F.Cu at (220.1, 76.6)
- added FB8: BLM18RK601SN1D, Resistors_SMD:R_0603, F.Cu at (189.9, 105.4)
- added FB9: BLM18RK601SN1D, Resistors_SMD:R_0603, F.Cu at (220.1, 71.6)
- added J1: USB_B_Micro, Connectors_USB:USB_Micro-B_Molex_47346-0001, F.Cu at (77.0, 79.0)
- added J2: USB_B_Micro, SMD_Packages:Conn-5, F.Cu at (148.6, 69.7)
- added J3: LiPo, Connectors_JST:JST_PH_S2B-PH-SM4-TB_02x2.00mm_Angled, F.Cu at (99.1, 53.5)
- added J4: USB_A, Connectors:USB_A, F.Cu at (90.8, 94.6)
- added J5: FFC-20, SMD_Packages:Conn-20, F.Cu at (166.0, 106.9)
- added J6: FFC-40, Connectors:HE10-40D, F.Cu at (144.2, 15.6)
- added L1: 6.8uH, Inductors_SMD:L_Taiyo-Yuden_NR-40xx_HandSoldering, F.Cu at (64.1, 68.1)
- added L2: BRL3225T150K, Resistors_SMD:R_1210, F.Cu at (108.0, 69.8)
- added Q1: MMUN2133LT1G, TO_SOT_Packages_SMD:SOT-23, F.Cu at (55.4, 64.8)
- added R101: 270K, Resistors_SMD:R_0402, F.Cu at (39.2, 72.1)
- added R102: 100K, Resistors_SMD:R_0402, F.Cu at (47.8, 62.3)
- added R103: 1K, Resistors_SMD:R_0402, F.Cu at (34.3, 67.7)
- added R104: 100K, Resistors_SMD:R_0402, F.Cu at (52.9, 57.0)
- added R105: 15K, Resistors_SMD:R_0402, F.Cu at (42.8, 67.2)
- added R106: 1.87M, Resistors_SMD:R_0402, F.Cu at (55.9, 72.1)
- added R107: 340K, Resistors_SMD:R_0402, F.Cu at (48.5, 57.0)
- added R108: 200K, Resistors_SMD:R_0402, F.Cu at (47.2, 67.2)
- added R109: 1.87M, Resistors_SMD:R_0402, F.Cu at (43.1, 62.4)
- added R110: 200K, Resistors_SMD:R_0402, F.Cu at (43.6, 72.1)
- added R111: 1K, Resistors_SMD:R_0402, F.Cu at (83.8, 49.8)
- added R112: 1K, Resistors_SMD:R_0402, F.Cu at (83.8, 55.4)
- added R113: 1K, Resistors_SMD:R_0402, F.Cu at (83.8, 52.3)
- added R201: 56K, Resistors_SMD:R_0402, F.Cu at (135.7, 162.7)
- added R202: 56K, Resistors_SMD:R_0402, F.Cu at (131.3, 165.0)
- added R203: 56K, Resistors_SMD:R_0402, F.Cu at (145.5, 154.7)
- added R204: 56K, Resistors_SMD:R_0402, F.Cu at (135.7, 167.5)
- added R301: 10K, Resistors_SMD:R_0402, F.Cu at (250.0, 72.3)
- added R302: 10K, Resistors_SMD:R_0402, F.Cu at (254.4, 72.3)
- added R303: 10K, Resistors_SMD:R_0402, F.Cu at (229.4, 96.8)
- added R304: 1K, Resistors_SMD:R_0402, F.Cu at (220.5, 104.8)
- added R305: 10K, Resistors_SMD:R_0402, F.Cu at (246.0, 78.0)
- added R306: 1K, Resistors_SMD:R_0402, F.Cu at (208.6, 100.3)
- added R307: 10K, Resistors_SMD:R_0402, F.Cu at (234.4, 66.5)
- added R308: 3, Resistors_SMD:R_0402, F.Cu at (199.8, 100.3)
- added R309: 12, Resistors_SMD:R_0402, F.Cu at (230.0, 66.5)
- added R310: 12, Resistors_SMD:R_0402, F.Cu at (204.2, 100.3)
- added SW1: SW_SPDT, Buttons_Switches_THT:SW_CuK_OS102011MA1QN1_SPDT_Angled, F.Cu at (81.3, 61.0)
- added U1: MCP73871, Housings_DFN_QFN:QFN-20-1EP_4x4mm_Pitch0.5mm, F.Cu at (96.8, 67.1)
- added U2: TPS61090, Housings_DFN_QFN:QFN-16-1EP_4x4mm_Pitch0.65mm, F.Cu at (108.0, 74.8)
- added U3: LM1117-3.3, TO_SOT_Packages_SMD:SOT-223-3_TabPin2, F.Cu at (146.9, 108.2)
- added U4: TFP401A, Housings_QFP:TQFP-100-1EP_14x14mm_Pitch0.5mm, F.Cu at (151.5, 90.9)
- added U5: 24LC02BT-OT, TO_SOT_Packages_SMD:TSOT-23-5, F.Cu at (217.3, 93.6)
- added U6: FAN5333, TO_SOT_Packages_SMD:SOT-23-5, F.Cu at (214.8, 101.9)
- added U7: AR1100-ISS, Housings_SOIC:SOIC-20W_7.5x12.8mm_Pitch1.27mm, F.Cu at (130.3, 84.1)
- added U8: USB2422, Housings_DFN_QFN:QFN-24-1EP_4x4mm_Pitch0.5mm, F.Cu at (116.6, 109.0)
- added Y1: 24M, Crystals:Crystal_SMD_0603-4pin_6.0x3.5mm, F.Cu at (139.7, 156.3)
- added Y2: 12M, Crystals:Resonator_SMD_muRata_CDSCB-2pin_4.5x2.0mm, F.Cu at (231.9, 85.0)
Other:
- copper layers 2 -> 4
